File: microsynth/Envelope.sch (KiCad schematic (older format))
At the start: 42 parts, among them IC5 TL074, Q3 BC548, SW18 SW_SPDT, SW19 SW_SPDT, SW20 SW_SPDT, SW7 SW_SPDT, SW8 SW_DPTT_SELECTOR, SW9 SW_DPTT_SELECTOR, U10 LM741, U3 4011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

Commit message: Footprints
Parts:
- U5: renamed from IC5; footprint (none) -> Package_DIP:DIP-14_W7.62mm
Changed lines of the file:
@@
 AR Path="/5E222DC1/5E7AFBE5" Ref="IC?"  Part="2"
 AR Path="/5E2BE1AD/5E7AFBE5" Ref="IC?"  Part="2"
-AR Path="/5E5B9865/5E7AFBE5" Ref="IC5"  Part="2"
-F 0 "IC5" H 10250 4017 50  0000 C CNN
+AR Path="/5E5B9865/5E7AFBE5" Ref="U5"  Part="2"
+F 0 "U5" H 10250 4017 50  0000 C CNN
 F 1 "TL074" H 10250 3926 50  0000 C CNN
-F 2 "" H 10200 3750 50  0001 C CNN
+F 2 "Package_DIP:DIP-14_W7.62mm" H 10200 3750 50  0001 C CNN
 F 3 "http://www.ti.com/lit/ds/symlink/tl071.pdf" H 10300 3850 50  0001 C CNN
 	2    10250 3650

Commit message: Footprints 2
Parts:
- C10, C11, C13, C14, C9: footprint (none) -> Capacitor_THT:C_Disc_D5.0mm_W2.5mm_P5.00mm
- C12: footprint (none) -> Capacitor_THT:CP_Radial_D10.0mm_P5.00mm; symbol Device:C -> Device:CP_Small
- D5: footprint (none) -> Diode_THT:D_A-405_P10.16mm_Horizontal
- Q3: footprint Package_TO_SOT_THT:TO-92_Inline -> Package_TO_SOT_THT:TO-92L_Inline_Wide
- SW8-SUSTAIN1: renamed from SW8; footprint (none) -> Button_Switch_THT:46313LDRX
- SW9: footprint (none) -> Button_Switch_THT:46313LDRX
- U10, U9: footprint (none) -> Package_DIP:DIP-8_W7.62mm_LongPads
- U3, U4, U8: footprint (none) -> Package_DIP:DIP-14_W7.62mm_LongPads
- renumbered RV10 to RV10-RELEASE1, RV12 to RV12-ENV-LEVEL1, RV9 to RV9-ATTACK1, SW18 to SW18-ENV-TO-VCF1, SW19 to SW19-ENV-TO-VCO1, SW20 to SW20-ENV-TO-KEYB1
Changed lines of the file:
@@
 F 0 "U4" H 4350 3627 50  0000 C CNN
 F 1 "4016" H 4350 3536 50  0000 C CNN
-F 2 "" H 4350 3800 50  0001 C CNN
+F 2 "Package_DIP:DIP-14_W7.62mm_LongPads" H 4350 3800 50  0001 C CNN
 F 3 "http://www.ti.com/lit/ds/symlink/cd4016b.pdf" H 4350 3800 50  0001 C CNN
 	2    4350 3800
@@
 F 0 "U4" H 4350 4227 50  0000 C CNN
 F 1 "4016" H 4350 4136 50  0000 C CNN
-F 2 "" H 4350 4400 50  0001 C CNN
+F 2 "Package_DIP:DIP-14_W7.62mm_LongPads" H 4350 4400 50  0001 C CNN
 F 3 "http://www.ti.com/lit/ds/symlink/cd4016b.pdf" H 4350 4400 50  0001 C CNN
 	3    4350 4400
@@
 F 0 "U4" H 9300 4127 50  0000 C CNN
 F 1 "4016" H 9300 4036 50  0000 C CNN
-F 2 "" H 9300 4300 50  0001 C CNN
+F 2 "Package_DIP:DIP-14_W7.62mm_LongPads" H 9300 4300 50  0001 C CNN
 F 3 "http://www.ti.com/lit/ds/symlink/cd4016b.pdf" H 9300 4300 50  0001 C CNN
 	4    9300 4300
@@
 F 0 "U4" H 9880 2096 50  0000 L CNN
 F 1 "4016" H 9880 2005 50  0000 L CNN
-F 2 "" H 9650 2050 50  0001 C CNN
+F 2 "Package_DIP:DIP-14_W7.62mm_LongPads" H 9650 2050 50  0001 C CNN
 F 3 "http://www.ti.com/lit/ds/symlink/cd4016b.pdf" H 9650 2050 50  0001 C CNN
 	5    9650 2050
@@
 F 0 "U8" H 1900 2275 50  0000 C CNN
 F 1 "4001" H 1900 2184 50  0000 C CNN
-F 2 "" H 1900 1950 50  0001 C CNN
+F 2 "Package_DIP:DIP-14_W7.62mm_LongPads" H 1900 1950 50  0001 C CNN
 F 3 "http://www.intersil.com/content/dam/Intersil/documents/cd40/cd4000bms-01bms-02bms-25bms.pdf" H 1900 1950 50  0001 C CNN
 	1    1900 1950
@@
 F 0 "U8" H 1900 2975 50  0000 C CNN
 F 1 "4001" H 1900 2884 50  0000 C CNN
-F 2 "" H 1900 2650 50  0001 C CNN
+F 2 "Package_DIP:DIP-14_W7.62mm_LongPads" H 1900 2650 50  0001 C CNN
 F 3 "http://www.intersil.com/content/dam/Intersil/documents/cd40/cd4000bms-01bms-02bms-25bms.pdf" H 1900 2650 50  0001 C CNN
 	2    1900 2650
@@
 F 0 "U8" H 1900 4225 50  0000 C CNN
 F 1 "4001" H 1900 4134 50  0000 C CNN
-F 2 "" H 1900 3900 50  0001 C CNN
+F 2 "Package_DIP:DIP-14_W7.62mm_LongPads" H 1900 3900 50  0001 C CNN
 F 3 "http://www.intersil.com/content/dam/Intersil/documents/cd40/cd4000bms-01bms-02bms-25bms.pdf" H 1900 3900 50  0001 C CNN
 	3    1900 3900
@@
 F 0 "U8" H 1850 3525 50  0000 C CNN
 F 1 "4001" H 1850 3434 50  0000 C CNN
-F 2 "" H 1850 3200 50  0001 C CNN
+F 2 "Package_DIP:DIP-14_W7.62mm_LongPads" H 1850 3200 50  0001 C CNN
 F 3 "http://www.intersil.com/content/dam/Intersil/documents/cd40/cd4000bms-01bms-02bms-25bms.pdf" H 1850 3200 50  0001 C CNN
 	4    1850 3200
@@
 F 0 "U8" H 9230 2096 50  0000 L CNN
 F 1 "4001" H 9230 2005 50  0000 L CNN
-F 2 "" H 9000 2050 50  0001 C CNN
+F 2 "Package_DIP:DIP-14_W7.62mm_LongPads" H 9000 2050 50  0001 C CNN
 F 3 "http://www.intersil.com/content/dam/Intersil/documents/cd40/cd4000bms-01bms-02bms-25bms.pdf" H 9000 2050 50  0001 C CNN
 	5    9000 2050
@@
 $Comp
 L Switch:SW_DPTT_SELECTOR SW?
-U 1 1 5E62FD95
+U 2 1 5E62FD95
 P 2950 3650
 AR Path="/5E475532/5E62FD95" Ref="SW?"  Part="1"
-AR Path="/5E5B9865/5E62FD95" Ref="SW8"  Part="1"
-F 0 "SW8" H 3144 3638 50  0000 L CNN
+AR Path="/5E5B9865/5E62FD95" Ref="SW8-SUSTAIN1"  Part="2"
+F 0 "SW8-SUSTAIN1" H 3144 3638 50  0000 L CNN
 F 1 "SW_DPTT_SELECTOR" H 3144 3547 50  0000 L CNN
-F 2 "" H 2950 3650 50  0001 C CNN
+F 2 "Button_Switch_THT:46313LDRX" H 2950 3650 50  0001 C CNN
 F 3 "" H 2950 3650 50  0001 C CNN
-	1    2950 3650
+	2    2950 3650
 	1    0    0    -1
 $EndComp
 $Comp
 L Switch:SW_DPTT_SELECTOR SW?
-U 2 1 5E62FD9B
+U 1 1 5E62FD9B
 P 2950 3550
 AR Path="/5E475532/5E62FD9B" Ref="SW?"  Part="2"
-AR Path="/5E5B9865/5E62FD9B" Ref="SW8"  Part="2"
-F 0 "SW8" H 3144 3679 50  0000 L CNN
+AR Path="/5E5B9865/5E62FD9B" Ref="SW8-SUSTAIN1"  Part="1"
+F 0 "SW8-SUSTAIN1" H 3144 3679 50  0000 L CNN
 F 1 "SW_DPTT_SELECTOR" H 3144 3588 50  0000 L CNN
-F 2 "" H 2950 3550 50  0001 C CNN
+F 2 "Button_Switch_THT:46313LDRX" H 2950 3550 50  0001 C CNN
 F 3 "" H 2950 3550 50  0001 C CNN
-	2    2950 3550
+	1    2950 3550
 	1    0    0    -1
 $EndComp
@@
 F 0 "C9" V 798 1850 50  0000 C CNN
 F 1 "10n" V 889 1850 50  0000 C CNN
-F 2 "" H 1088 1700 50  0001 C CNN
+F 2 "Capacitor_THT:C_Disc_D5.0mm_W2.5mm_P5.00mm" H 1088 1700 50  0001 C CNN
 F 3 "~" H 1050 1850 50  0001 C CNN
 	1    1050 1850
@@
 F 0 "C10" V 798 3100 50  0000 C CNN
 F 1 "10n" V 889 3100 50  0000 C CNN
-F 2 "" H 1088 2950 50  0001 C CNN
+F 2 "Capacitor_THT:C_Disc_D5.0mm_W2.5mm_P5.00mm" H 1088 2950 50  0001 C CNN
 F 3 "~" H 1050 3100 50  0001 C CNN
 	1    1050 3100
@@
 F 0 "C13" V 8398 4300 50  0000 C CNN
 F 1 "10n" V 8489 4300 50  0000 C CNN
-F 2 "" H 8688 4150 50  0001 C CNN
+F 2 "Capacitor_THT:C_Disc_D5.0mm_W2.5mm_P5.00mm" H 8688 4150 50  0001 C CNN
 F 3 "~" H 8650 4300 50  0001 C CNN
 	1    8650 4300
@@
 $EndComp
 $Comp
-L Device:R_POT RV10
+L Device:R_POT RV10-RELEASE1
 U 1 1 5E666B6F
 P 4350 4900
-F 0 "RV10" H 4280 4946 50  0000 R CNN
+F 0 "RV10-RELEASE1" H 4280 4946 50  0000 R CNN
 F 1 "2MLOG" H 4280 4855 50  0000 R CNN
 F 2 "" H 4350 4900 50  0001 C CNN
@@
 $EndComp
 $Comp
-L Device:R_POT RV9
+L Device:R_POT RV9-ATTACK1
 U 1 1 5E66825F
 P 4350 3300
-F 0 "RV9" H 4280 3346 50  0000 R CNN
+F 0 "RV9-ATTACK1" H 4280 3346 50  0000 R CNN
 F 1 "1MLOG" H 4280 3255 50  0000 R CNN
 F 2 "" H 4350 3300 50  0001 C CNN
@@
 Connection ~ 4350 4100
 $Comp
-L Device:C C12
+L Device:CP_Small C12
 U 1 1 5E675EDC
 P 5150 4350
 F 0 "C12" H 5265 4396 50  0000 L CNN
 F 1 "4.7u" H 5265 4305 50  0000 L CNN
-F 2 "" H 5188 4200 50  0001 C CNN
+F 2 "Capacitor_THT:CP_Radial_D10.0mm_P5.00mm" H 5188 4200 50  0001 C CNN
 F 3 "~" H 5150 4350 50  0001 C CNN
 	1    5150 4350
 	1    0    0    -1
 $EndComp
-Wire Wire Line
-	5150 4200 5150 4100
 Connection ~ 5150 4100
-Wire Wire Line
-	5150 4500 5150 5150
 Connection ~ 5150 5150
 $Comp
@@
 F 0 "U9" H 6294 3204 50  0000 L CNN
 F 1 "LM741" H 6294 3295 50  0000 L CNN
-F 2 "" H 6000 3300 50  0001 C CNN
+F 2 "Package_DIP:DIP-8_W7.62mm_LongPads" H 6000 3300 50  0001 C CNN
 F 3 "http://www.ti.com/lit/ds/symlink/lm741.pdf" H 6100 3400 50  0001 C CNN
 	1    5950 3250
@@
 F 0 "U10" H 6294 4604 50  0000 L CNN
 F 1 "LM741" H 6294 4695 50  0000 L CNN
-F 2 "" H 6000 4700 50  0001 C CNN
+F 2 "Package_DIP:DIP-8_W7.62mm_LongPads" H 6000 4700 50  0001 C CNN
 F 3 "http://www.ti.com/lit/ds/symlink/lm741.pdf" H 6100 4800 50  0001 C CNN
 	1    5950 4650
@@
 F 0 "Q3" H 3941 4796 50  0000 L CNN
 F 1 "BC548" H 3941 4705 50  0000 L CNN
-F 2 "Package_TO_SOT_THT:TO-92_Inline" H 3950 4675 50  0001 L CIN
+F 2 "Package_TO_SOT_THT:TO-92L_Inline_Wide" H 3950 4675 50  0001 L CIN
 F 3 "http://www.fairchildsemi.com/ds/BC/BC547.pdf" H 3750 4750 50  0001 L CNN
 	1    3750 4750
@@
 F 0 "C11" H 3415 1996 50  0000 L CNN
 F 1 "1u" H 3415 1905 50  0000 L CNN
-F 2 "" H 3338 1800 50  0001 C CNN
+F 2 "Capacitor_THT:C_Disc_D5.0mm_W2.5mm_P5.00mm" H 3338 1800 50  0001 C CNN
 F 3 "~" H 3300 1950 50  0001 C CNN
 	1    3300 1950
@@
 F 0 "D5" H 1400 1766 50  0000 C CNN
 F 1 "OA81" H 1400 1675 50  0000 C CNN
-F 2 "" H 1400 1550 50  0001 C CNN
+F 2 "Diode_THT:D_A-405_P10.16mm_Horizontal" H 1400 1550 50  0001 C CNN
 F 3 "~" H 1400 1550 50  0001 C CNN
 	1    1400 1550
@@
 	5600 3100 5600 2750
 $Comp
-L Device:R_POT RV12
+L Device:R_POT RV12-ENV-LEVEL1
 U 1 1 5E71BB7F
 P 6650 3550
-F 0 "RV12" H 6580 3596 50  0000 R CNN
+F 0 "RV12-ENV-LEVEL1" H 6580 3596 50  0000 R CNN
 F 1 "100k" H 6580 3505 50  0000 R CNN
 F 2 "" H 6650 3550 50  0001 C CNN
@@
 F 0 "SW9" H 7894 4833 50  0000 L CNN
 F 1 "SW_DPTT_SELECTOR" H 7894 4742 50  0000 L CNN
-F 2 "" H 7700 4800 50  0001 C CNN
+F 2 "Button_Switch_THT:46313LDRX" H 7700 4800 50  0001 C CNN
 F 3 "" H 7700 4800 50  0001 C CNN
 F 4 "TRIGGER" H 7894 4651 50  0000 L CNN "Label"
@@
 F 0 "C14" H 9715 3896 50  0000 L CNN
 F 1 "100n" H 9715 3805 50  0000 L CNN
-F 2 "" H 9638 3700 50  0001 C CNN
+F 2 "Capacitor_THT:C_Disc_D5.0mm_W2.5mm_P5.00mm" H 9638 3700 50  0001 C CNN
 F 3 "~" H 9600 3850 50  0001 C CNN
 	1    9600 3850
@@
 F 0 "U3" H 8700 4175 50  0000 C CNN
 F 1 "4011" H 8700 4084 50  0000 C CNN
-F 2 "" H 8700 3850 50  0001 C CNN
+F 2 "Package_DIP:DIP-14_W7.62mm_LongPads" H 8700 3850 50  0001 C CNN
 F 3 "http://www.intersil.com/content/dam/Intersil/documents/cd40/cd4011bms-12bms-23bms.pdf" H 8700 3850 50  0001 C CNN
 	4    8700 3850
@@
 F 0 "U3" H 8000 4175 50  0000 C CNN
 F 1 "4011" H 8000 4084 50  0000 C CNN
-F 2 "" H 8000 3850 50  0001 C CNN
+F 2 "Package_DIP:DIP-14_W7.62mm_LongPads" H 8000 3850 50  0001 C CNN
 F 3 "http://www.intersil.com/content/dam/Intersil/documents/cd40/cd4011bms-12bms-23bms.pdf" H 8000 3850 50  0001 C CNN
 	3    8000 3850
@@
 	8300 4300 7200 4300
 $Comp
-L Switch:SW_SPDT SW20
+L Switch:SW_SPDT SW20-ENV-TO-KEYB1
 U 1 1 5E83D5A9
 P 7750 1000
-F 0 "SW20" H 7750 1285 50  0000 C CNN
+F 0 "SW20-ENV-TO-KEYB1" H 7750 1285 50  0000 C CNN
 F 1 "SW_SPDT" H 7750 1194 50  0000 C CNN
 F 2 "" H 7750 1000 50  0001 C CNN
@@
 	7400 2600 7600 2600
 $Comp
-L Switch:SW_SPDT SW19
+L Switch:SW_SPDT SW19-ENV-TO-VCO1
 U 1 1 5E85AAE1
 P 7750 1700
-F 0 "SW19" H 7750 1985 50  0000 C CNN
+F 0 "SW19-ENV-TO-VCO1" H 7750 1985 50  0000 C CNN
 F 1 "SW_SPDT" H 7750 1894 50  0000 C CNN
 F 2 "" H 7750 1700 50  0001 C CNN
@@
 	7400 1700 7400 2400
 $Comp
-L Switch:SW_SPDT SW18
+L Switch:SW_SPDT SW18-ENV-TO-VCF1
 U 1 1 5E881667
 P 7750 2400
-F 0 "SW18" H 7750 2685 50  0000 C CNN
+F 0 "SW18-ENV-TO-VCF1" H 7750 2685 50  0000 C CNN
 F 1 "SW_SPDT" H 7750 2594 50  0000 C CNN
 F 2 "" H 7750 2400 50  0001 C CNN
@@
 Wire Wire Line
 	4350 5150 5150 5150
+Wire Wire Line
+	5150 4100 5150 4250
+Wire Wire Line
+	5150 4450 5150 5150
 $EndSCHEMATC

Commit message: Hacking together the footprints
Parts:
- RV10-RELEASE1, RV9-ATTACK1: footprint (none) -> 4ms_Potentiometer:Pot_16mm_NoDet_RV16AF-4A
- RV11: footprint (none) -> Potentiometers:Potentiometer_Trimmer_Bourns_PV36W
- RV12-ENV-LEVEL1: value 100k -> 100kLIN; footprint (none) -> 4ms_Potentiometer:Pot_16mm_NoDet_RV16AF-4A
- SW18-ENV-TO-VCF1, SW19-ENV-TO-VCO1, SW20-ENV-TO-KEYB1, SW7: footprint (none) -> 4ms:SPDT_KIT
- SW8-SUSTAIN1, SW9: footprint Button_Switch_THT:46313LDRX -> Buttons_Switches_ThroughHole:DP3T_Toggle; symbol Switch:SW_DPTT_SELECTOR -> microsynth-rescue:SW_DPTT_SELECTOR-Switch
Changed lines of the file:
@@
 $EndComp
 $Comp
-L Switch:SW_DPTT_SELECTOR SW?
+L microsynth-rescue:SW_DPTT_SELECTOR-Switch SW?
 U 2 1 5E62FD95
-P 2950 3650
+P 2950 3550
 AR Path="/5E475532/5E62FD95" Ref="SW?"  Part="1"
 AR Path="/5E5B9865/5E62FD95" Ref="SW8-SUSTAIN1"  Part="2"
-F 0 "SW8-SUSTAIN1" H 3144 3638 50  0000 L CNN
-F 1 "SW_DPTT_SELECTOR" H 3144 3547 50  0000 L CNN
-F 2 "Button_Switch_THT:46313LDRX" H 2950 3650 50  0001 C CNN
-F 3 "" H 2950 3650 50  0001 C CNN
-	2    2950 3650
-	1    0    0    -1
-$EndComp
-$Comp
-L Switch:SW_DPTT_SELECTOR SW?
+AR Path="/5E62FD95" Ref="SW8-SUSTAIN1"  Part="2"
+F 0 "SW8-SUSTAIN1" H 3144 3538 50  0000 L CNN
+F 1 "SW_DPTT_SELECTOR" H 3144 3447 50  0000 L CNN
+F 2 "Buttons_Switches_ThroughHole:DP3T_Toggle" H 2950 3550 50  0001 C CNN
+F 3 "" H 2950 3550 50  0001 C CNN
+	2    2950 3550
+	1    0    0    -1
+$EndComp
+$Comp
+L microsynth-rescue:SW_DPTT_SELECTOR-Switch SW?
 U 1 1 5E62FD9B
-P 2950 3550
+P 2950 3650
 AR Path="/5E475532/5E62FD9B" Ref="SW?"  Part="2"
 AR Path="/5E5B9865/5E62FD9B" Ref="SW8-SUSTAIN1"  Part="1"
-F 0 "SW8-SUSTAIN1" H 3144 3679 50  0000 L CNN
-F 1 "SW_DPTT_SELECTOR" H 3144 3588 50  0000 L CNN
-F 2 "Button_Switch_THT:46313LDRX" H 2950 3550 50  0001 C CNN
-F 3 "" H 2950 3550 50  0001 C CNN
-	1    2950 3550
+AR Path="/5E62FD9B" Ref="SW8-SUSTAIN1"  Part="1"
+F 0 "SW8-SUSTAIN1" H 3144 3779 50  0000 L CNN
+F 1 "SW_DPTT_SELECTOR" H 3144 3688 50  0000 L CNN
+F 2 "Buttons_Switches_ThroughHole:DP3T_Toggle" H 2950 3650 50  0001 C CNN
+F 3 "" H 2950 3650 50  0001 C CNN
+	1    2950 3650
 	1    0    0    -1
 $EndComp
@@
 F 0 "RV11" H 6580 4646 50  0000 R CNN
 F 1 "100k" H 6580 4555 50  0000 R CNN
-F 2 "" H 6650 4600 50  0001 C CNN
+F 2 "Potentiometers:Potentiometer_Trimmer_Bourns_PV36W" H 6650 4600 50  0001 C CNN
 F 3 "~" H 6650 4600 50  0001 C CNN
 	1    6650 4600
@@
 F 0 "RV10-RELEASE1" H 4280 4946 50  0000 R CNN
 F 1 "2MLOG" H 4280 4855 50  0000 R CNN
-F 2 "" H 4350 4900 50  0001 C CNN
+F 2 "4ms_Potentiometer:Pot_16mm_NoDet_RV16AF-4A" H 4350 4900 50  0001 C CNN
 F 3 "~" H 4350 4900 50  0001 C CNN
 	1    4350 4900
@@
 F 0 "RV9-ATTACK1" H 4280 3346 50  0000 R CNN
 F 1 "1MLOG" H 4280 3255 50  0000 R CNN
-F 2 "" H 4350 3300 50  0001 C CNN
+F 2 "4ms_Potentiometer:Pot_16mm_NoDet_RV16AF-4A" H 4350 3300 50  0001 C CNN
 F 3 "~" H 4350 3300 50  0001 C CNN
 	1    4350 3300
@@
 F 0 "SW7" V 3859 1712 50  0000 R CNN
 F 1 "SW_SPDT" V 3950 1712 50  0000 R CNN
-F 2 "" H 3950 1900 50  0001 C CNN
+F 2 "4ms:SPDT_KIT" H 3950 1900 50  0001 C CNN
 F 3 "~" H 3950 1900 50  0001 C CNN
 F 4 "ADSR" V 4041 1712 50  0000 R CNN "Label"
@@
 P 6650 3550
 F 0 "RV12-ENV-LEVEL1" H 6580 3596 50  0000 R CNN
-F 1 "100k" H 6580 3505 50  0000 R CNN
-F 2 "" H 6650 3550 50  0001 C CNN
+F 1 "100kLIN" H 6580 3505 50  0000 R CNN
+F 2 "4ms_Potentiometer:Pot_16mm_NoDet_RV16AF-4A" H 6650 3550 50  0001 C CNN
 F 3 "~" H 6650 3550 50  0001 C CNN
 	1    6650 3550
@@
 	7600 2600 7600 2650
 $Comp
-L Switch:SW_DPTT_SELECTOR SW9
+L microsynth-rescue:SW_DPTT_SELECTOR-Switch SW9
 U 1 1 5E74BE8F
 P 7700 4800
+AR Path="/5E74BE8F" Ref="SW9"  Part="1"
+AR Path="/5E5B9865/5E74BE8F" Ref="SW9"  Part="1"
 F 0 "SW9" H 7894 4833 50  0000 L CNN
 F 1 "SW_DPTT_SELECTOR" H 7894 4742 50  0000 L CNN
-F 2 "Button_Switch_THT:46313LDRX" H 7700 4800 50  0001 C CNN
+F 2 "Buttons_Switches_ThroughHole:DP3T_Toggle" H 7700 4800 50  0001 C CNN
 F 3 "" H 7700 4800 50  0001 C CNN
 F 4 "TRIGGER" H 7894 4651 50  0000 L CNN "Label"
@@
 F 0 "SW20-ENV-TO-KEYB1" H 7750 1285 50  0000 C CNN
 F 1 "SW_SPDT" H 7750 1194 50  0000 C CNN
-F 2 "" H 7750 1000 50  0001 C CNN
+F 2 "4ms:SPDT_KIT" H 7750 1000 50  0001 C CNN
 F 3 "~" H 7750 1000 50  0001 C CNN
 	1    7750 1000
@@
 F 0 "SW19-ENV-TO-VCO1" H 7750 1985 50  0000 C CNN
 F 1 "SW_SPDT" H 7750 1894 50  0000 C CNN
-F 2 "" H 7750 1700 50  0001 C CNN
+F 2 "4ms:SPDT_KIT" H 7750 1700 50  0001 C CNN
 F 3 "~" H 7750 1700 50  0001 C CNN
 	1    7750 1700
@@
 F 0 "SW18-ENV-TO-VCF1" H 7750 2685 50  0000 C CNN
 F 1 "SW_SPDT" H 7750 2594 50  0000 C CNN
-F 2 "" H 7750 2400 50  0001 C CNN
+F 2 "4ms:SPDT_KIT" H 7750 2400 50  0001 C CNN
 F 3 "~" H 7750 2400 50  0001 C CNN
 	1    7750 2400

Commit message: All components placed on PCB
Parts:
- C11: footprint Capacitor_THT:C_Disc_D5.0mm_W2.5mm_P5.00mm -> Capacitor_THT:CP_Radial_D5.0mm_P2.50mm; symbol Device:C -> Device:CP_Small
- C12: footprint Capacitor_THT:CP_Radial_D10.0mm_P5.00mm -> Capacitor_THT:CP_Radial_D5.0mm_P2.50mm
- SW9: value SW_DPTT_SELECTOR -> SW_DPTT_SELECTOR-Switch; Label TRIGGER -> (none)
Changed lines of the file:
@@
 F 0 "C12" H 5265 4396 50  0000 L CNN
 F 1 "4.7u" H 5265 4305 50  0000 L CNN
-F 2 "Capacitor_THT:CP_Radial_D10.0mm_P5.00mm" H 5188 4200 50  0001 C CNN
+F 2 "Capacitor_THT:CP_Radial_D5.0mm_P2.50mm" H 5188 4200 50  0001 C CNN
 F 3 "~" H 5150 4350 50  0001 C CNN
 	1    5150 4350
@@
 Connection ~ 2950 2150
 $Comp
-L Device:C C11
+L Device:CP_Small C11
 U 1 1 5E6D9634
-P 3300 1950
-F 0 "C11" H 3415 1996 50  0000 L CNN
-F 1 "1u" H 3415 1905 50  0000 L CNN
-F 2 "Capacitor_THT:C_Disc_D5.0mm_W2.5mm_P5.00mm" H 3338 1800 50  0001 C CNN
-F 3 "~" H 3300 1950 50  0001 C CNN
-	1    3300 1950
+P 3300 1900
+F 0 "C11" H 3415 1946 50  0000 L CNN
+F 1 "1u" H 3415 1855 50  0000 L CNN
+F 2 "Capacitor_THT:CP_Radial_D5.0mm_P2.50mm" H 3338 1750 50  0001 C CNN
+F 3 "~" H 3300 1900 50  0001 C CNN
+	1    3300 1900
 	1    0    0    -1
 $EndComp
@@
 L power:-VSW #PWR0190
 U 1 1 5E6D9EA0
-P 3300 2200
-F 0 "#PWR0190" H 3300 2300 50  0001 C CNN
-F 1 "-VSW" H 3315 2373 50  0000 C CNN
-F 2 "" H 3300 2200 50  0001 C CNN
-F 3 "" H 3300 2200 50  0001 C CNN
-	1    3300 2200
+P 3300 2100
+F 0 "#PWR0190" H 3300 2200 50  0001 C CNN
+F 1 "-VSW" H 3315 2273 50  0000 C CNN
+F 2 "" H 3300 2100 50  0001 C CNN
+F 3 "" H 3300 2100 50  0001 C CNN
+	1    3300 2100
 	-1   0    0    1
 $EndComp
 Wire Wire Line
-	3300 2200 3300 2100
+	3300 2100 3300 2000
 Wire Wire Line
 	3300 1800 3300 1700
@@
 Wire Wire Line
 	7600 2600 7600 2650
-$Comp
-L microsynth-rescue:SW_DPTT_SELECTOR-Switch SW9
-U 1 1 5E74BE8F
-P 7700 4800
-AR Path="/5E74BE8F" Ref="SW9"  Part="1"
-AR Path="/5E5B9865/5E74BE8F" Ref="SW9"  Part="1"
-F 0 "SW9" H 7894 4833 50  0000 L CNN
-F 1 "SW_DPTT_SELECTOR" H 7894 4742 50  0000 L CNN
-F 2 "Buttons_Switches_ThroughHole:DP3T_Toggle" H 7700 4800 50  0001 C CNN
-F 3 "" H 7700 4800 50  0001 C CNN
-F 4 "TRIGGER" H 7894 4651 50  0000 L CNN "Label"
-	1    7700 4800
-	1    0    0    -1
-$EndComp
 NoConn ~ 7550 5000
 NoConn ~ 7850 5000
@@
 Wire Wire Line
 	8300 4300 7200 4300
-$Comp
-L Switch:SW_SPDT SW20-ENV-TO-KEYB1
-U 1 1 5E83D5A9
-P 7750 1000
-F 0 "SW20-ENV-TO-KEYB1" H 7750 1285 50  0000 C CNN
-F 1 "SW_SPDT" H 7750 1194 50  0000 C CNN
-F 2 "4ms:SPDT_KIT" H 7750 1000 50  0001 C CNN
-F 3 "~" H 7750 1000 50  0001 C CNN
-	1    7750 1000
-	1    0    0    -1
-$EndComp
 Wire Wire Line
 	8050 1100 7950 1100
@@
 Wire Wire Line
 	5150 4450 5150 5150
+$Comp
+L microsynth-rescue:SW_DPTT_SELECTOR-Switch SW9
+U 1 1 5E95BE3D
+P 7700 4800
+F 0 "SW9" H 7900 4800 50  0000 L CNN
+F 1 "SW_DPTT_SELECTOR-Switch" H 7900 4700 50  0000 L CNN
+F 2 "Buttons_Switches_ThroughHole:DP3T_Toggle" H 7700 4800 50  0001 C CNN
+F 3 "" H 7700 4800 50  0001 C CNN
+	1    7700 4800
+	1    0    0    -1
+$EndComp
+$Comp
+L Switch:SW_SPDT SW20-ENV-TO-KEYB1
+U 1 1 5E83D5A9
+P 7750 1000
+F 0 "SW20-ENV-TO-KEYB1" H 7750 1285 50  0000 C CNN
+F 1 "SW_SPDT" H 7750 1194 50  0000 C CNN
+F 2 "4ms:SPDT_KIT" H 7750 1000 50  0001 C CNN
+F 3 "~" H 7750 1000 50  0001 C CNN
+	1    7750 1000
+	1    0    0    -1
+$EndComp
 $EndSCHEMATC
