File: microsynth/Envelope.sch (KiCad schematic (older format))
At the start: 42 parts, among them Q3 BC548, SW18-ENV-TO-VCF1 SW_SPDT, SW19-ENV-TO-VCO1 SW_SPDT, SW20-ENV-TO-KEYB1 SW_SPDT, SW7 SW_SPDT, SW8-SUSTAIN1 SW_DPTT_SELECTOR, SW9 SW_DPTT_SELECTOR-Switch, U10 LM741, U3 4011, U4 4016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

Commit message: Laying out pcb
Parts:
- removed SW8-SUSTAIN1: SW_DPTT_SELECTOR, Buttons_Switches_ThroughHole:DP3T_Toggle, symbol microsynth-rescue:SW_DPTT_SELECTOR-Switch
- removed U5: TL074, Package_DIP:DIP-14_W7.62mm, symbol Amplifier_Operational:TL074
- added SW8: SW_DPTT_SELECTOR-Switch, Buttons_Switches_ThroughHole:DP3T_Toggle, symbol Switch:SW_DPTT_SELECTOR-Switch
- added unit 5 of U3
- added U5: LF347, Package_DIP:DIP-14_W7.62mm_LongPads, symbol Amplifier_Operational:LF347
- RV10: renamed from RV10-RELEASE1; Label (none) -> Release
- RV12: renamed from RV12-ENV-LEVEL1; Label (none) -> Env Level
- RV9: renamed from RV9-ATTACK1; Label (none) -> Attack
- SW9: value SW_DPTT_SELECTOR-Switch -> TRIGGER
Connections:
- net +VSW: now also SW8.2, SW8.4, SW8.7, U3.14 (VDD)
- net -VSW: now also U3.7 (VSS)
- net TO_D3: now also U8.13; no longer U8.12
- net TO_S12_THUMBWEEL: now also U5.6 (-), U5.7
- net TO_VCA_R136: now also SW8.8
- net at C12.1, R62.1, U4.4: now also U4.8; no longer U4.9
- net at RV10.1, RV10.2: now also U4.9; no longer U4.8
- net at C14.1, U4.11: now also U5.5 (+)
- net at U8.10: now also U8.12, SW8.3; no longer U8.13
- net at U8.8: now also RV11.2; no longer U8.11
- net at U8.9: now also U8.11; no longer RV11.2
- net at C10.2, C9.2, D5.1 (K)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: now also SW8.1
Changed lines of the file:
@@
 F 3 "http://www.ti.com/lit/ds/symlink/cd4016b.pdf" H 4350 4400 50  0001 C CNN
 	3    4350 4400
-	0    -1   -1   0
+	0    -1   1    0
 $EndComp
 $Comp
@@
 U 3 1 5E5BF1E4
 P 1900 3900
-F 0 "U8" H 1900 4225 50  0000 C CNN
-F 1 "4001" H 1900 4134 50  0000 C CNN
+F 0 "U8" H 1900 3900 50  0000 C CNN
+F 1 "4001" H 1900 3700 50  0000 C CNN
 F 2 "Package_DIP:DIP-14_W7.62mm_LongPads" H 1900 3900 50  0001 C CNN
 F 3 "http://www.intersil.com/content/dam/Intersil/documents/cd40/cd4000bms-01bms-02bms-25bms.pdf" H 1900 3900 50  0001 C CNN
 	3    1900 3900
-	1    0    0    -1
+	1    0    0    1
 $EndComp
 $Comp
@@
 U 4 1 5E5BFBC6
 P 1850 3200
-F 0 "U8" H 1850 3525 50  0000 C CNN
-F 1 "4001" H 1850 3434 50  0000 C CNN
+F 0 "U8" H 1850 3200 50  0000 C CNN
+F 1 "4001" H 1850 3000 50  0000 C CNN
 F 2 "Package_DIP:DIP-14_W7.62mm_LongPads" H 1850 3200 50  0001 C CNN
 F 3 "http://www.intersil.com/content/dam/Intersil/documents/cd40/cd4000bms-01bms-02bms-25bms.pdf" H 1850 3200 50  0001 C CNN
 	4    1850 3200
-	1    0    0    -1
+	1    0    0    1
 $EndComp
 $Comp
@@
 F 3 "http://www.intersil.com/content/dam/Intersil/documents/cd40/cd4000bms-01bms-02bms-25bms.pdf" H 9000 2050 50  0001 C CNN
 	5    9000 2050
-	1    0    0    -1
-$EndComp
-$Comp
-L microsynth-rescue:SW_DPTT_SELECTOR-Switch SW?
-U 2 1 5E62FD95
-P 2950 3550
-AR Path="/5E475532/5E62FD95" Ref="SW?"  Part="1"
-AR Path="/5E5B9865/5E62FD95" Ref="SW8-SUSTAIN1"  Part="2"
-AR Path="/5E62FD95" Ref="SW8-SUSTAIN1"  Part="2"
-F 0 "SW8-SUSTAIN1" H 3144 3538 50  0000 L CNN
-F 1 "SW_DPTT_SELECTOR" H 3144 3447 50  0000 L CNN
-F 2 "Buttons_Switches_ThroughHole:DP3T_Toggle" H 2950 3550 50  0001 C CNN
-F 3 "" H 2950 3550 50  0001 C CNN
-	2    2950 3550
-	1    0    0    -1
-$EndComp
-$Comp
-L microsynth-rescue:SW_DPTT_SELECTOR-Switch SW?
-U 1 1 5E62FD9B
-P 2950 3650
-AR Path="/5E475532/5E62FD9B" Ref="SW?"  Part="2"
-AR Path="/5E5B9865/5E62FD9B" Ref="SW8-SUSTAIN1"  Part="1"
-AR Path="/5E62FD9B" Ref="SW8-SUSTAIN1"  Part="1"
-F 0 "SW8-SUSTAIN1" H 3144 3779 50  0000 L CNN
-F 1 "SW_DPTT_SELECTOR" H 3144 3688 50  0000 L CNN
-F 2 "Buttons_Switches_ThroughHole:DP3T_Toggle" H 2950 3650 50  0001 C CNN
-F 3 "" H 2950 3650 50  0001 C CNN
-	1    2950 3650
 	1    0    0    -1
 $EndComp
@@
 $EndComp
 $Comp
-L Device:R_POT RV10-RELEASE1
+L Device:R_POT RV10
 U 1 1 5E666B6F
 P 4350 4900
-F 0 "RV10-RELEASE1" H 4280 4946 50  0000 R CNN
+F 0 "RV10" H 4280 4946 50  0000 R CNN
 F 1 "2MLOG" H 4280 4855 50  0000 R CNN
 F 2 "4ms_Potentiometer:Pot_16mm_NoDet_RV16AF-4A" H 4350 4900 50  0001 C CNN
 F 3 "~" H 4350 4900 50  0001 C CNN
+F 4 "Release" H 4100 4750 50  0000 C BNN "Label"
 	1    4350 4900
 	1    0    0    -1
 $EndComp
 $Comp
-L Device:R_POT RV9-ATTACK1
+L Device:R_POT RV9
 U 1 1 5E66825F
 P 4350 3300
-F 0 "RV9-ATTACK1" H 4280 3346 50  0000 R CNN
+F 0 "RV9" H 4280 3346 50  0000 R CNN
 F 1 "1MLOG" H 4280 3255 50  0000 R CNN
 F 2 "4ms_Potentiometer:Pot_16mm_NoDet_RV16AF-4A" H 4350 3300 50  0001 C CNN
 F 3 "~" H 4350 3300 50  0001 C CNN
+F 4 "Attack" H 4150 3150 50  0000 C CNN "Label"
 	1    4350 3300
 	1    0    0    -1
@@
 	5600 3100 5600 2750
 $Comp
-L Device:R_POT RV12-ENV-LEVEL1
+L Device:R_POT RV12
 U 1 1 5E71BB7F
 P 6650 3550
-F 0 "RV12-ENV-LEVEL1" H 6580 3596 50  0000 R CNN
+F 0 "RV12" H 6580 3596 50  0000 R CNN
 F 1 "100kLIN" H 6580 3505 50  0000 R CNN
 F 2 "4ms_Potentiometer:Pot_16mm_NoDet_RV16AF-4A" H 6650 3550 50  0001 C CNN
 F 3 "~" H 6650 3550 50  0001 C CNN
+F 4 "Env Level" H 6550 3450 50  0000 R TNN "Label"
 	1    6650 3550
 	1    0    0    -1
@@
 	1    0    0    -1
 $EndComp
-$Comp
-L power:-VSW #PWR0195
-U 1 1 5E8A3AFC
-P 9650 2550
-F 0 "#PWR0195" H 9650 2650 50  0001 C CNN
-F 1 "-VSW" H 9665 2723 50  0000 C CNN
-F 2 "" H 9650 2550 50  0001 C CNN
-F 3 "" H 9650 2550 50  0001 C CNN
-	1    9650 2550
-	-1   0    0    1
-$EndComp
 Wire Wire Line
 	4200 1100 4600 1100
@@
 	1    5850 4950
 	-1   0    0    1
-$EndComp
-$Comp
-L Amplifier_Operational:TL074 IC?
-U 2 1 5E7AFBE5
-P 10250 3650
-AR Path="/5E222DC1/5E7AFBE5" Ref="IC?"  Part="2"
-AR Path="/5E2BE1AD/5E7AFBE5" Ref="IC?"  Part="2"
-AR Path="/5E5B9865/5E7AFBE5" Ref="U5"  Part="2"
-F 0 "U5" H 10250 4017 50  0000 C CNN
-F 1 "TL074" H 10250 3926 50  0000 C CNN
-F 2 "Package_DIP:DIP-14_W7.62mm" H 10200 3750 50  0001 C CNN
-F 3 "http://www.ti.com/lit/ds/symlink/tl071.pdf" H 10300 3850 50  0001 C CNN
-	2    10250 3650
-	1    0    0    -1
 $EndComp
 Text GLabel 8050 1100 2    50   BiDi ~ 0
@@
 P 7700 4800
 F 0 "SW9" H 7900 4800 50  0000 L CNN
-F 1 "SW_DPTT_SELECTOR-Switch" H 7900 4700 50  0000 L CNN
+F 1 "TRIGGER" H 7900 4700 50  0000 L CNN
 F 2 "Buttons_Switches_ThroughHole:DP3T_Toggle" H 7700 4800 50  0001 C CNN
 F 3 "" H 7700 4800 50  0001 C CNN
@@
 	1    0    0    -1
 $EndComp
+$Comp
+L Amplifier_Operational:LF347 U?
+U 2 1 5E8FB113
+P 10250 3650
+AR Path="/5E8C1704/5E8FB113" Ref="U?"  Part="2"
+AR Path="/5E5B9865/5E8FB113" Ref="U5"  Part="2"
+F 0 "U5" H 10250 4050 50  0000 C CNN
+F 1 "LF347" H 10250 3950 50  0000 C CNN
+F 2 "Package_DIP:DIP-14_W7.62mm_LongPads" H 10200 3750 50  0001 C CNN
+F 3 "https://www.ti.com/lit/ds/symlink/lf147.pdf" H 10300 3850 50  0001 C CNN
+	2    10250 3650
+	1    0    0    -1
+$EndComp
+$Comp
+L 4xxx:4011 U3
+U 5 1 5EBF5D48
+P 10350 2050
+F 0 "U3" H 10600 2100 50  0000 L CNN
+F 1 "4011" H 10600 2050 50  0000 L CNN
+F 2 "Package_DIP:DIP-14_W7.62mm_LongPads" H 10350 2050 50  0001 C CNN
+F 3 "http://www.intersil.com/content/dam/Intersil/documents/cd40/cd4011bms-12bms-23bms.pdf" H 10350 2050 50  0001 C CNN
+	5    10350 2050
+	1    0    0    -1
+$EndComp
+$Comp
+L power:-VSW #PWR0195
+U 1 1 5E8A3AFC
+P 9650 2550
+F 0 "#PWR0195" H 9650 2650 50  0001 C CNN
+F 1 "-VSW" H 9665 2723 50  0000 C CNN
+F 2 "" H 9650 2550 50  0001 C CNN
+F 3 "" H 9650 2550 50  0001 C CNN
+	1    9650 2550
+	-1   0    0    1
+$EndComp
+$Comp
+L power:-VSW #PWR0149
+U 1 1 5EC0045E
+P 10350 2550
+F 0 "#PWR0149" H 10350 2650 50  0001 C CNN
+F 1 "-VSW" H 10365 2723 50  0000 C CNN
+F 2 "" H 10350 2550 50  0001 C CNN
+F 3 "" H 10350 2550 50  0001 C CNN
+	1    10350 2550
+	-1   0    0    1
+$EndComp
+$Comp
+L power:+VSW #PWR0150
+U 1 1 5EC00B84
+P 10350 1550
+F 0 "#PWR0150" H 10350 1400 50  0001 C CNN
+F 1 "+VSW" H 10365 1723 50  0000 C CNN
+F 2 "" H 10350 1550 50  0001 C CNN
+F 3 "" H 10350 1550 50  0001 C CNN
+	1    10350 1550
+	1    0    0    -1
+$EndComp
+$Comp
+L Switch:SW_DPTT_SELECTOR-Switch SW8
+U 1 1 5F2DEA06
+P 2950 3650
+F 0 "SW8" H 3200 3650 50  0000 L CNN
+F 1 "SW_DPTT_SELECTOR-Switch" H 3200 3550 50  0000 L CNN
+F 2 "Buttons_Switches_ThroughHole:DP3T_Toggle" H 2950 3650 50  0001 C CNN
+F 3 "" H 2950 3650 50  0001 C CNN
+	1    2950 3650
+	1    0    0    -1
+$EndComp
+$Comp
+L Switch:SW_DPTT_SELECTOR-Switch SW8
+U 2 1 5F2DFAB2
+P 2950 3550
+F 0 "SW8" H 3200 3750 50  0000 L CNN
+F 1 "SW_DPTT_SELECTOR-Switch" H 3200 3650 50  0000 L CNN
+F 2 "Buttons_Switches_ThroughHole:DP3T_Toggle" H 2950 3550 50  0001 C CNN
+F 3 "" H 2950 3550 50  0001 C CNN
+F 4 "Sustain" H 3200 3550 50  0000 L CNN "Label"
+	2    2950 3550
+	1    0    0    -1
+$EndComp

Commit message: Laying out pcb ...
Connections:
- net +VSW: no longer R61.2, SW8.2, SW8.4, U4.5
- new net: R61.2, SW8.2, SW8.4, U4.5
Changed lines of the file:
@@
 Wire Wire Line
 	3850 3050 3850 3300
-Wire Wire Line
-	4050 3800 3850 3800
-Connection ~ 3850 3800
-Wire Wire Line
-	3850 3800 3850 3950
 $Comp
 L power:+VSW #PWR0188
@@
 $EndComp
 Wire Wire Line
-	3400 3800 3850 3800
-Wire Wire Line
 	3400 3950 3400 3800
 Wire Wire Line
@@
 	3000 3300 3850 3300
 Connection ~ 3850 3300
-Wire Wire Line
-	3850 3300 3850 3800
 Wire Wire Line
 	3100 3350 3500 3350
@@
 	1    0    0    -1
 $EndComp
+Wire Wire Line
+	3400 3800 4050 3800
+Wire Wire Line
+	3850 3300 3850 3950
 $EndSCHEMATC
