File: microsynth/Keyboard.sch (KiCad schematic (older format))
At the start: 51 parts, among them IC5 TL074, Q1 BC182, Q2 BC182L, SW1 SW_DPTT_SELECTOR, SW9 SW_DPTT_SELECTOR, U1 TL074, U2 TL072, U3 4011, U4 4016, U6 TL071

Commit message: Footprints
Parts:
- U5: renamed from IC5; footprint (none) -> Package_DIP:DIP-14_W7.62mm
Changed lines of the file:
@@
 AR Path="/5E222DC1/5E8D0FAD" Ref="IC?"  Part="1"
 AR Path="/5E2BE1AD/5E8D0FAD" Ref="IC?"  Part="1"
-AR Path="/5E8C1704/5E8D0FAD" Ref="IC5"  Part="1"
-F 0 "IC5" H 6100 2617 50  0000 C CNN
+AR Path="/5E8C1704/5E8D0FAD" Ref="U5"  Part="1"
+F 0 "U5" H 6100 2617 50  0000 C CNN
 F 1 "TL074" H 6100 2526 50  0000 C CNN
-F 2 "" H 6050 2350 50  0001 C CNN
+F 2 "Package_DIP:DIP-14_W7.62mm" H 6050 2350 50  0001 C CNN
 F 3 "http://www.ti.com/lit/ds/symlink/tl071.pdf" H 6150 2450 50  0001 C CNN
 	1    6100 2250
@@
 U 4 1 5EAFC72E
 P 5550 3300
-F 0 "U1" H 5550 2933 50  0000 C CNN
-F 1 "TL074" H 5550 3024 50  0000 C CNN
+F 0 "U1" H 5550 3300 50  0000 C CNN
+F 1 "TL074" H 5600 3500 50  0000 C CNN
 F 2 "Package_DIP:DIP-14_W7.62mm" H 5500 3400 50  0001 C CNN
 F 3 "http://www.ti.com/lit/ds/symlink/tl071.pdf" H 5600 3500 50  0001 C CNN
@@
 U 3 1 5EB1727D
 P 5500 3950
-F 0 "U1" H 5500 3583 50  0000 C CNN
+F 0 "U1" H 5500 3950 50  0000 C CNN
 F 1 "TL074" H 5500 3674 50  0000 C CNN
 F 2 "Package_DIP:DIP-14_W7.62mm" H 5450 4050 50  0001 C CNN

Commit message: Footprints 2
Parts:
- added J6, J7: Conn_01x02_Male, Connector_PinHeader_2.54mm:PinHeader_1x02_P2.54mm_Vertical, symbol Connector:Conn_01x02_Male
- C1, C2, C3, C4, C5, C6, C7: footprint (none) -> Capacitor_THT:C_Disc_D5.0mm_W2.5mm_P5.00mm
- Q1, Q2: footprint (none) -> Package_TO_SOT_THT:TO-92L_Inline_Wide
- RV1-TUNE1: renamed from RV1; footprint (none) -> Potentiometer_THT:Potentiometer_Omeg_PC16BU_Vertical
- RV2-GLIDE1: renamed from RV2; footprint (none) -> Potentiometer_THT:Potentiometer_Omeg_PC16BU_Vertical
- RV3-SCALE1: renamed from RV3; footprint (none) -> Potentiometer_THT:Potentiometer_Omeg_PC16BU_Vertical
- SW1: footprint (none) -> Button_Switch_THT:46313LDRX
- SW1-DRIFT1: renamed from SW1; footprint (none) -> Button_Switch_THT:46313LDRX
- SW9-TRIGGER1: renamed from SW9; footprint (none) -> Button_Switch_THT:46313LDRX
- U2, U6: footprint (none) -> Package_DIP:DIP-8_W7.62mm_LongPads
- U3, U4: footprint (none) -> Package_DIP:DIP-14_W7.62mm_LongPads
Other:
- moved on the sheet: U4A
Changed lines of the file:
@@
 F 0 "Q2" H 10791 2454 50  0000 L CNN
 F 1 "BC182L" H 10791 2545 50  0000 L CNN
-F 2 "" H 10800 2600 50  0001 C CNN
+F 2 "Package_TO_SOT_THT:TO-92L_Inline_Wide" H 10800 2600 50  0001 C CNN
 F 3 "~" H 10600 2500 50  0001 C CNN
 	1    10600 2500
@@
 F 0 "Q1" H 9491 1554 50  0000 L CNN
 F 1 "BC182" H 9491 1645 50  0000 L CNN
-F 2 "" H 9500 1700 50  0001 C CNN
+F 2 "Package_TO_SOT_THT:TO-92L_Inline_Wide" H 9500 1700 50  0001 C CNN
 F 3 "~" H 9300 1600 50  0001 C CNN
 	1    9300 1600
@@
 F 0 "C6" H 9815 1696 50  0000 L CNN
 F 1 "10n" H 9815 1605 50  0000 L CNN
-F 2 "" H 9738 1500 50  0001 C CNN
+F 2 "Capacitor_THT:C_Disc_D5.0mm_W2.5mm_P5.00mm" H 9738 1500 50  0001 C CNN
 F 3 "~" H 9700 1650 50  0001 C CNN
 	1    9700 1650
@@
 F 0 "C7" H 10215 2946 50  0000 L CNN
 F 1 "100n" H 10215 2855 50  0000 L CNN
-F 2 "" H 10138 2750 50  0001 C CNN
+F 2 "Capacitor_THT:C_Disc_D5.0mm_W2.5mm_P5.00mm" H 10138 2750 50  0001 C CNN
 F 3 "~" H 10100 2900 50  0001 C CNN
 	1    10100 2900
@@
 F 0 "C5" V 7548 2700 50  0000 C CNN
 F 1 "470n" V 7639 2700 50  0000 C CNN
-F 2 "" H 7838 2550 50  0001 C CNN
+F 2 "Capacitor_THT:C_Disc_D5.0mm_W2.5mm_P5.00mm" H 7838 2550 50  0001 C CNN
 F 3 "~" H 7800 2700 50  0001 C CNN
 	1    7800 2700
@@
 F 0 "C4" H 6515 2896 50  0000 L CNN
 F 1 "100n" H 6515 2805 50  0000 L CNN
-F 2 "" H 6438 2700 50  0001 C CNN
+F 2 "Capacitor_THT:C_Disc_D5.0mm_W2.5mm_P5.00mm" H 6438 2700 50  0001 C CNN
 F 3 "~" H 6400 2850 50  0001 C CNN
 	1    6400 2850
@@
 F 0 "C1" H 5715 2746 50  0000 L CNN
 F 1 "1u" H 5715 2655 50  0000 L CNN
-F 2 "" H 5638 2550 50  0001 C CNN
+F 2 "Capacitor_THT:C_Disc_D5.0mm_W2.5mm_P5.00mm" H 5638 2550 50  0001 C CNN
 F 3 "~" H 5600 2700 50  0001 C CNN
 	1    5600 2700
@@
 F 0 "C2" V 798 1900 50  0000 C CNN
 F 1 "22n" V 889 1900 50  0000 C CNN
-F 2 "" H 1088 1750 50  0001 C CNN
+F 2 "Capacitor_THT:C_Disc_D5.0mm_W2.5mm_P5.00mm" H 1088 1750 50  0001 C CNN
 F 3 "~" H 1050 1900 50  0001 C CNN
 	1    1050 1900
@@
 F 0 "U3" H 2450 3125 50  0000 C CNN
 F 1 "4011" H 2450 3034 50  0000 C CNN
-F 2 "" H 2450 2800 50  0001 C CNN
+F 2 "Package_DIP:DIP-14_W7.62mm_LongPads" H 2450 2800 50  0001 C CNN
 F 3 "http://www.intersil.com/content/dam/Intersil/documents/cd40/cd4011bms-12bms-23bms.pdf" H 2450 2800 50  0001 C CNN
 	1    2450 2800
@@
 F 0 "U3" H 3050 3125 50  0000 C CNN
 F 1 "4011" H 3050 3034 50  0000 C CNN
-F 2 "" H 3050 2800 50  0001 C CNN
+F 2 "Package_DIP:DIP-14_W7.62mm_LongPads" H 3050 2800 50  0001 C CNN
 F 3 "http://www.intersil.com/content/dam/Intersil/documents/cd40/cd4011bms-12bms-23bms.pdf" H 3050 2800 50  0001 C CNN
 	2    3050 2800
@@
 Connection ~ 3350 2800
 $Comp
-L Switch:SW_DPTT_SELECTOR SW9
-U 2 1 5E8EB5AF
+L Switch:SW_DPTT_SELECTOR SW9-TRIGGER1
+U 1 1 5E8EB5AF
 P 2550 3700
-F 0 "SW9" H 2744 3874 50  0000 L CNN
+F 0 "SW9-TRIGGER1" H 2744 3874 50  0000 L CNN
 F 1 "SW_DPTT_SELECTOR" H 2744 3783 50  0000 L CNN
-F 2 "" H 2550 3700 50  0001 C CNN
+F 2 "Button_Switch_THT:46313LDRX" H 2550 3700 50  0001 C CNN
 F 3 "" H 2550 3700 50  0001 C CNN
 F 4 "TRIGGER" H 2744 3692 50  0000 L CNN "Label"
-	2    2550 3700
+	1    2550 3700
 	1    0    0    -1
 $EndComp
@@
 L 4xxx:4016 U4
 U 1 1 5E903589
-P 5000 1750
-F 0 "U4" H 5000 1485 50  0000 C CNN
-F 1 "4016" H 5000 1576 50  0000 C CNN
-F 2 "" H 5000 1750 50  0001 C CNN
-F 3 "http://www.ti.com/lit/ds/symlink/cd4016b.pdf" H 5000 1750 50  0001 C CNN
-	1    5000 1750
+P 5000 1900
+F 0 "U4" H 5000 1635 50  0000 C CNN
+F 1 "4016" H 5000 1726 50  0000 C CNN
+F 2 "Package_DIP:DIP-14_W7.62mm_LongPads" H 5000 1900 50  0001 C CNN
+F 3 "http://www.ti.com/lit/ds/symlink/cd4016b.pdf" H 5000 1900 50  0001 C CNN
+	1    5000 1900
 	-1   0    0    1
 $EndComp
 Wire Wire Line
-	5000 2050 5000 2300
+	5000 2200 5000 2300
 Wire Wire Line
 	5000 2300 2150 2300
@@
 Connection ~ 2150 2600
 Wire Wire Line
-	5600 2150 5600 1750
-Wire Wire Line
-	5600 1750 5300 1750
+	5600 2150 5600 1900
+Wire Wire Line
+	5600 1900 5300 1900
 Connection ~ 5600 2150
 $Comp
@@
 TO_R2
 Wire Wire Line
-	1550 1300 1300 1300
-Wire Wire Line
 	1300 1300 1300 1050
-Text Label 4600 1250 2    50   ~ 0
+Text Label 4600 1300 2    50   ~ 0
 TO_R27
-Wire Wire Line
-	4600 1250 4700 1250
-Wire Wire Line
-	4700 1250 4700 950
 Wire Wire Line
 	4700 950  1900 950
@@
 	4850 1250 4950 1250
 $Comp
-L Switch:SW_DPTT_SELECTOR SW1
+L Switch:SW_DPTT_SELECTOR SW1-DRIFT1
 U 1 1 5E91DC50
 P 5650 1050
-F 0 "SW1" H 5844 1083 50  0000 L CNN
+F 0 "SW1-DRIFT1" H 5844 1083 50  0000 L CNN
 F 1 "SW_DPTT_SELECTOR" H 5844 992 50  0000 L CNN
-F 2 "" H 5650 1050 50  0001 C CNN
+F 2 "Button_Switch_THT:46313LDRX" H 5650 1050 50  0001 C CNN
 F 3 "" H 5650 1050 50  0001 C CNN
 F 4 "DRIFT" H 5844 901 50  0000 L CNN "Label"
@@
 Wire Wire Line
 	5600 1250 5600 1400
-Connection ~ 5600 1750
+Connection ~ 5600 1900
 Wire Wire Line
 	5500 1250 5250 1250
@@
 Connection ~ 5600 1400
 Wire Wire Line
-	5600 1400 5600 1750
+	5600 1400 5600 1900
 $Comp
 L Device:R R32
@@
 F 0 "SW1" H 5844 1079 50  0000 L CNN
 F 1 "SW_DPTT_SELECTOR" H 5844 988 50  0000 L CNN
-F 2 "" H 5650 950 50  0001 C CNN
+F 2 "Button_Switch_THT:46313LDRX" H 5650 950 50  0001 C CNN
 F 3 "" H 5650 950 50  0001 C CNN
 	2    5650 950
@@
 	7000 1800 7000 1700
 $Comp
-L Device:R_POT RV1
+L Device:R_POT RV1-TUNE1
 U 1 1 5E936F79
 P 7000 1150
-F 0 "RV1" V 6793 1150 50  0000 C CNN
+F 0 "RV1-TUNE1" V 6793 1150 50  0000 C CNN
 F 1 "100k" V 6884 1150 50  0000 C CNN
-F 2 "" H 7000 1150 50  0001 C CNN
+F 2 "Potentiometer_THT:Potentiometer_Omeg_PC16BU_Vertical" H 7000 1150 50  0001 C CNN
 F 3 "~" H 7000 1150 50  0001 C CNN
 	1    7000 1150
@@
 $EndComp
 $Comp
-L Device:R_POT_TRIM RV3
+L Device:R_POT_TRIM RV3-SCALE1
 U 1 1 5E974C22
 P 9550 2500
-F 0 "RV3" V 9435 2500 50  0000 C CNN
+F 0 "RV3-SCALE1" V 9435 2500 50  0000 C CNN
 F 1 "22K" V 9344 2500 50  0000 C CNN
-F 2 "" H 9550 2500 50  0001 C CNN
+F 2 "Potentiometer_THT:Potentiometer_Omeg_PC16BU_Vertical" H 9550 2500 50  0001 C CNN
 F 3 "~" H 9550 2500 50  0001 C CNN
 F 4 "SCALE" V 9253 2500 50  0000 C CNN "Label"
@@
 	7400 2700 7650 2700
 $Comp
-L Device:R_POT RV2
+L Device:R_POT RV2-GLIDE1
 U 1 1 5EA28367
 P 7950 2350
-F 0 "RV2" V 7835 2350 50  0000 C CNN
+F 0 "RV2-GLIDE1" V 7835 2350 50  0000 C CNN
 F 1 "2MLOG" V 7744 2350 50  0000 C CNN
-F 2 "" H 7950 2350 50  0001 C CNN
+F 2 "Potentiometer_THT:Potentiometer_Omeg_PC16BU_Vertical" H 7950 2350 50  0001 C CNN
 F 3 "~" H 7950 2350 50  0001 C CNN
 F 4 "GLIDE" V 7653 2350 50  0000 C CNN "Label"
@@
 F 0 "C3" H 4865 2796 50  0000 L CNN
 F 1 "100u" H 4865 2705 50  0000 L CNN
-F 2 "" H 4788 2600 50  0001 C CNN
+F 2 "Capacitor_THT:C_Disc_D5.0mm_W2.5mm_P5.00mm" H 4788 2600 50  0001 C CNN
 F 3 "~" H 4750 2750 50  0001 C CNN
 	1    4750 2750
@@
 Text Label 1450 1900 0    50   ~ 0
 TO_KEYBOARD_CONTACTS
-Wire Wire Line
-	1450 1900 1300 1900
 Connection ~ 1300 1900
-Wire Wire Line
-	4450 1750 4700 1750
 Wire Wire Line
 	8350 2400 8300 2400
@@
 F 0 "U6" H 8994 2546 50  0000 L CNN
 F 1 "TL071" H 8994 2455 50  0000 L CNN
-F 2 "" H 8700 2550 50  0001 C CNN
+F 2 "Package_DIP:DIP-8_W7.62mm_LongPads" H 8700 2550 50  0001 C CNN
 F 3 "http://www.ti.com/lit/ds/symlink/tl071.pdf" H 8800 2650 50  0001 C CNN
 	1    8650 2500
@@
 F 0 "U2" H 10100 883 50  0000 C CNN
 F 1 "TL072" H 10100 974 50  0000 C CNN
-F 2 "" H 10100 1250 50  0001 C CNN
+F 2 "Package_DIP:DIP-8_W7.62mm_LongPads" H 10100 1250 50  0001 C CNN
 F 3 "http://www.ti.com/lit/ds/symlink/tl071.pdf" H 10100 1250 50  0001 C CNN
 	2    10100 1250
@@
 F 0 "U2" H 7350 2717 50  0000 C CNN
 F 1 "TL072" H 7350 2626 50  0000 C CNN
-F 2 "" H 7350 2350 50  0001 C CNN
+F 2 "Package_DIP:DIP-8_W7.62mm_LongPads" H 7350 2350 50  0001 C CNN
 F 3 "http://www.ti.com/lit/ds/symlink/tl071.pdf" H 7350 2350 50  0001 C CNN
 	1    7350 2350
@@
 Wire Wire Line
 	10700 2700 10700 3050
-Text GLabel 4450 1750 0    50   BiDi ~ 0
-FROM_KEYBOARD_CONTACTS
 Text GLabel 8850 3550 0    50   BiDi ~ 0
 TO_R41
@@
 Text GLabel 8900 3100 0    50   BiDi ~ 0
 VIN_TO_SEQ_SKT
+$Comp
+L Connector:Conn_01x02_Male J6
+U 1 1 5E83A10F
+P 3100 1100
+F 0 "J6" V 3162 1144 50  0000 L CNN
+F 1 "Conn_01x02_Male" V 3253 1144 50  0000 L CNN
+F 2 "Connector_PinHeader_2.54mm:PinHeader_1x02_P2.54mm_Vertical" H 3100 1100 50  0001 C CNN
+F 3 "~" H 3100 1100 50  0001 C CNN
+	1    3100 1100
+	0    1    1    0
+$EndComp
+Wire Wire Line
+	1300 1300 3000 1300
+Wire Wire Line
+	3100 1300 4700 1300
+Wire Wire Line
+	4700 950  4700 1300
+$Comp
+L Connector:Conn_01x02_Male J7
+U 1 1 5E864311
+P 3100 1700
+F 0 "J7" V 3162 1744 50  0000 L CNN
+F 1 "Conn_01x02_Male" V 3253 1744 50  0000 L CNN
+F 2 "Connector_PinHeader_2.54mm:PinHeader_1x02_P2.54mm_Vertical" H 3100 1700 50  0001 C CNN
+F 3 "~" H 3100 1700 50  0001 C CNN
+	1    3100 1700
+	0    1    1    0
+$EndComp
+Wire Wire Line
+	1300 1900 3000 1900
+Wire Wire Line
+	4700 1900 3100 1900
+Text Label 4700 1900 2    50   ~ 0
+FROM_KEYBOARD_CONTACTS
 $EndSCHEMATC

Commit message: Hacking together the footprints
Parts:
- RV1-TUNE1, RV3-SCALE1: footprint Potentiometer_THT:Potentiometer_Omeg_PC16BU_Vertical -> Potentiometers:Potentiometer_Trimmer_Bourns_PV36W
- RV2-GLIDE1: footprint Potentiometer_THT:Potentiometer_Omeg_PC16BU_Vertical -> 4ms_Potentiometer:Pot_16mm_NoDet_RV16AF-4A
- SW1, SW1-DRIFT1, SW9-TRIGGER1: footprint Button_Switch_THT:46313LDRX -> Buttons_Switches_ThroughHole:DP3T_Toggle; symbol Switch:SW_DPTT_SELECTOR -> microsynth-rescue:SW_DPTT_SELECTOR-Switch
Changed lines of the file:
@@
 	3350 3150 3300 3150
 Connection ~ 3350 2800
-$Comp
-L Switch:SW_DPTT_SELECTOR SW9-TRIGGER1
-U 1 1 5E8EB5AF
-P 2550 3700
-F 0 "SW9-TRIGGER1" H 2744 3874 50  0000 L CNN
-F 1 "SW_DPTT_SELECTOR" H 2744 3783 50  0000 L CNN
-F 2 "Button_Switch_THT:46313LDRX" H 2550 3700 50  0001 C CNN
-F 3 "" H 2550 3700 50  0001 C CNN
-F 4 "TRIGGER" H 2744 3692 50  0000 L CNN "Label"
-	1    2550 3700
-	1    0    0    -1
-$EndComp
 Wire Wire Line
 	2400 3500 2400 3300
@@
 	4850 1250 4950 1250
 $Comp
-L Switch:SW_DPTT_SELECTOR SW1-DRIFT1
+L microsynth-rescue:SW_DPTT_SELECTOR-Switch SW1-DRIFT1
 U 1 1 5E91DC50
 P 5650 1050
+AR Path="/5E91DC50" Ref="SW1-DRIFT1"  Part="1"
+AR Path="/5E8C1704/5E91DC50" Ref="SW1-DRIFT1"  Part="1"
 F 0 "SW1-DRIFT1" H 5844 1083 50  0000 L CNN
 F 1 "SW_DPTT_SELECTOR" H 5844 992 50  0000 L CNN
-F 2 "Button_Switch_THT:46313LDRX" H 5650 1050 50  0001 C CNN
+F 2 "Buttons_Switches_ThroughHole:DP3T_Toggle" H 5650 1050 50  0001 C CNN
 F 3 "" H 5650 1050 50  0001 C CNN
 F 4 "DRIFT" H 5844 901 50  0000 L CNN "Label"
@@
 	6100 1250 5800 1250
 $Comp
-L Switch:SW_DPTT_SELECTOR SW1
+L microsynth-rescue:SW_DPTT_SELECTOR-Switch SW1
 U 2 1 5E929054
 P 5650 950
+AR Path="/5E929054" Ref="SW1"  Part="2"
+AR Path="/5E8C1704/5E929054" Ref="SW1"  Part="2"
 F 0 "SW1" H 5844 1079 50  0000 L CNN
 F 1 "SW_DPTT_SELECTOR" H 5844 988 50  0000 L CNN
-F 2 "Button_Switch_THT:46313LDRX" H 5650 950 50  0001 C CNN
+F 2 "Buttons_Switches_ThroughHole:DP3T_Toggle" H 5650 950 50  0001 C CNN
 F 3 "" H 5650 950 50  0001 C CNN
 	2    5650 950
@@
 F 0 "RV1-TUNE1" V 6793 1150 50  0000 C CNN
 F 1 "100k" V 6884 1150 50  0000 C CNN
-F 2 "Potentiometer_THT:Potentiometer_Omeg_PC16BU_Vertical" H 7000 1150 50  0001 C CNN
+F 2 "Potentiometers:Potentiometer_Trimmer_Bourns_PV36W" H 7000 1150 50  0001 C CNN
 F 3 "~" H 7000 1150 50  0001 C CNN
 	1    7000 1150
@@
 F 0 "RV3-SCALE1" V 9435 2500 50  0000 C CNN
 F 1 "22K" V 9344 2500 50  0000 C CNN
-F 2 "Potentiometer_THT:Potentiometer_Omeg_PC16BU_Vertical" H 9550 2500 50  0001 C CNN
+F 2 "Potentiometers:Potentiometer_Trimmer_Bourns_PV36W" H 9550 2500 50  0001 C CNN
 F 3 "~" H 9550 2500 50  0001 C CNN
 F 4 "SCALE" V 9253 2500 50  0000 C CNN "Label"
@@
 F 0 "RV2-GLIDE1" V 7835 2350 50  0000 C CNN
 F 1 "2MLOG" V 7744 2350 50  0000 C CNN
-F 2 "Potentiometer_THT:Potentiometer_Omeg_PC16BU_Vertical" H 7950 2350 50  0001 C CNN
+F 2 "4ms_Potentiometer:Pot_16mm_NoDet_RV16AF-4A" H 7950 2350 50  0001 C CNN
 F 3 "~" H 7950 2350 50  0001 C CNN
 F 4 "GLIDE" V 7653 2350 50  0000 C CNN "Label"
@@
 Text Label 4700 1900 2    50   ~ 0
 FROM_KEYBOARD_CONTACTS
+$Comp
+L microsynth-rescue:SW_DPTT_SELECTOR-Switch SW9-TRIGGER1
+U 1 1 5E8EB5AF
+P 2550 3700
+AR Path="/5E8EB5AF" Ref="SW9-TRIGGER1"  Part="1"
+AR Path="/5E8C1704/5E8EB5AF" Ref="SW9-TRIGGER1"  Part="1"
+F 0 "SW9-TRIGGER1" H 2744 3874 50  0000 L CNN
+F 1 "SW_DPTT_SELECTOR" H 2744 3783 50  0000 L CNN
+F 2 "Buttons_Switches_ThroughHole:DP3T_Toggle" H 2550 3700 50  0001 C CNN
+F 3 "" H 2550 3700 50  0001 C CNN
+F 4 "TRIGGER" H 2744 3692 50  0000 L CNN "Label"
+	1    2550 3700
+	-1   0    0    1
+$EndComp
 $EndSCHEMATC

Commit message: All components placed on PCB
Parts:
- removed SW1, SW9-TRIGGER1: SW_DPTT_SELECTOR, Buttons_Switches_ThroughHole:DP3T_Toggle, symbol microsynth-rescue:SW_DPTT_SELECTOR-Switch
- added R2: 680, Resistor_THT:R_Axial_DIN0207_L6.3mm_D2.5mm_P10.16mm_Horizontal, symbol Device:R
- added R27: 1k2, Resistor_THT:R_Axial_DIN0207_L6.3mm_D2.5mm_P10.16mm_Horizontal, symbol Device:R
- added SW9: SW_DPTT_SELECTOR-Switch, Buttons_Switches_ThroughHole:DP3T_Toggle, symbol microsynth-rescue:SW_DPTT_SELECTOR-Switch
- C3: footprint Capacitor_THT:C_Disc_D5.0mm_W2.5mm_P5.00mm -> Capacitor_THT:CP_Radial_D5.0mm_P2.50mm; symbol Device:C -> Device:CP_Small
Connections:
- net +VSW: now also SW9.6
- net TO_S9A_KEYBOARD_CONTROLLER: now also SW9.8
- net at U3.2: now also SW9.5, SW9.7
- net TO_R2: no longer names the net of R1.1, U1.6 (-)
- net TO_R2: now also R2.2; no longer J6.2 (Pin_2)
- net TO_R27: no longer names the net of J6.1 (Pin_1)
- net TO_R27: now also R27.2; no longer U1.7
- new net: J6.2 (Pin_2), R2.1
- new net: R27.1, U1.7
- no-connect marks 6 -> 2
Changed lines of the file:
@@
 F 3 "~" H 7800 2700 50  0001 C CNN
 	1    7800 2700
-	0    1    1    0
+	0    1    -1   0
 $EndComp
 $Comp
@@
 AR Path="/5E2BE1AD/5E8D0FAD" Ref="IC?"  Part="1"
 AR Path="/5E8C1704/5E8D0FAD" Ref="U5"  Part="1"
-F 0 "U5" H 6100 2617 50  0000 C CNN
+F 0 "U5" H 6050 2250 50  0000 C CNN
 F 1 "TL074" H 6100 2526 50  0000 C CNN
 F 2 "Package_DIP:DIP-14_W7.62mm" H 6050 2350 50  0001 C CNN
@@
 Wire Wire Line
 	800  1050 800  1250
-Text Label 1550 1300 0    50   ~ 0
-TO_R2
 Wire Wire Line
 	1300 1300 1300 1050
-Text Label 4600 1300 2    50   ~ 0
-TO_R27
 Wire Wire Line
 	4700 950  1900 950
@@
 F 3 "~" H 6250 1250 50  0001 C CNN
 	1    6250 1250
-	0    1    1    0
+	0    1    -1   0
 $EndComp
 Wire Wire Line
 	6100 1250 5800 1250
-$Comp
-L microsynth-rescue:SW_DPTT_SELECTOR-Switch SW1
-U 2 1 5E929054
-P 5650 950
-AR Path="/5E929054" Ref="SW1"  Part="2"
-AR Path="/5E8C1704/5E929054" Ref="SW1"  Part="2"
-F 0 "SW1" H 5844 1079 50  0000 L CNN
-F 1 "SW_DPTT_SELECTOR" H 5844 988 50  0000 L CNN
-F 2 "Buttons_Switches_ThroughHole:DP3T_Toggle" H 5650 950 50  0001 C CNN
-F 3 "" H 5650 950 50  0001 C CNN
-	2    5650 950
-	1    0    0    -1
-$EndComp
-NoConn ~ 5500 750
-NoConn ~ 5600 750
-NoConn ~ 5700 750
-NoConn ~ 5800 750
 $Comp
 L power:-VSW #PWR0208
@@
 L power:-VSW #PWR0218
 U 1 1 5EA46F8D
-P 4750 3000
-F 0 "#PWR0218" H 4750 3100 50  0001 C CNN
-F 1 "-VSW" H 4765 3173 50  0000 C CNN
-F 2 "" H 4750 3000 50  0001 C CNN
-F 3 "" H 4750 3000 50  0001 C CNN
-	1    4750 3000
+P 4750 2800
+F 0 "#PWR0218" H 4750 2900 50  0001 C CNN
+F 1 "-VSW" H 4765 2973 50  0000 C CNN
+F 2 "" H 4750 2800 50  0001 C CNN
+F 3 "" H 4750 2800 50  0001 C CNN
+	1    4750 2800
 	-1   0    0    1
 $EndComp
 $Comp
-L Device:C C3
+L Device:CP_Small C3
 U 1 1 5EA4781A
-P 4750 2750
-F 0 "C3" H 4865 2796 50  0000 L CNN
-F 1 "100u" H 4865 2705 50  0000 L CNN
-F 2 "Capacitor_THT:C_Disc_D5.0mm_W2.5mm_P5.00mm" H 4788 2600 50  0001 C CNN
-F 3 "~" H 4750 2750 50  0001 C CNN
-	1    4750 2750
-	1    0    0    -1
-$EndComp
-Wire Wire Line
-	4750 2900 4750 3000
-Wire Wire Line
-	4750 2600 4750 2500
+P 4750 2650
+F 0 "C3" H 4865 2696 50  0000 L CNN
+F 1 "100u" H 4865 2605 50  0000 L CNN
+F 2 "Capacitor_THT:CP_Radial_D5.0mm_P2.50mm" H 4788 2500 50  0001 C CNN
+F 3 "~" H 4750 2650 50  0001 C CNN
+	1    4750 2650
+	1    0    0    -1
+$EndComp
+Wire Wire Line
+	4750 2750 4750 2800
+Wire Wire Line
+	4750 2550 4750 2500
 Text Label 1450 1900 0    50   ~ 0
 TO_KEYBOARD_CONTACTS
@@
 U 1 1 5EA6B0F3
 P 8650 2500
-F 0 "U6" H 8994 2546 50  0000 L CNN
-F 1 "TL071" H 8994 2455 50  0000 L CNN
+F 0 "U6" H 8550 2500 50  0000 L CNN
+F 1 "TL071" H 8650 2650 50  0000 L CNN
 F 2 "Package_DIP:DIP-8_W7.62mm_LongPads" H 8700 2550 50  0001 C CNN
 F 3 "http://www.ti.com/lit/ds/symlink/tl071.pdf" H 8800 2650 50  0001 C CNN
@@
 U 2 1 5EA9A5A0
 P 10100 1250
-F 0 "U2" H 10100 883 50  0000 C CNN
+F 0 "U2" H 10050 1250 50  0000 C CNN
 F 1 "TL072" H 10100 974 50  0000 C CNN
 F 2 "Package_DIP:DIP-8_W7.62mm_LongPads" H 10100 1250 50  0001 C CNN
@@
 U 1 1 5EAE7191
 P 7350 2350
-F 0 "U2" H 7350 2717 50  0000 C CNN
-F 1 "TL072" H 7350 2626 50  0000 C CNN
+F 0 "U2" H 7300 2350 50  0000 C CNN
+F 1 "TL072" H 7400 2550 50  0000 C CNN
 F 2 "Package_DIP:DIP-8_W7.62mm_LongPads" H 7350 2350 50  0001 C CNN
 F 3 "http://www.ti.com/lit/ds/symlink/tl071.pdf" H 7350 2350 50  0001 C CNN
@@
 U 1 1 5EB303DC
 P 1700 2600
-F 0 "U1" H 1700 2967 50  0000 C CNN
+F 0 "U1" H 1650 2600 50  0000 C CNN
 F 1 "TL074" H 1700 2876 50  0000 C CNN
 F 2 "Package_DIP:DIP-14_W7.62mm" H 1650 2700 50  0001 C CNN
@@
 U 2 1 5EB34716
 P 1600 950
-F 0 "U1" H 1600 1317 50  0000 C CNN
+F 0 "U1" H 1550 950 50  0000 C CNN
 F 1 "TL074" H 1600 1226 50  0000 C CNN
 F 2 "Package_DIP:DIP-14_W7.62mm" H 1550 1050 50  0001 C CNN
@@
 $EndComp
 Wire Wire Line
-	1300 1300 3000 1300
-Wire Wire Line
-	3100 1300 4700 1300
+	1300 1300 1650 1300
+Wire Wire Line
+	3100 1300 4100 1300
 Wire Wire Line
 	4700 950  4700 1300
@@
 FROM_KEYBOARD_CONTACTS
 $Comp
-L microsynth-rescue:SW_DPTT_SELECTOR-Switch SW9-TRIGGER1
-U 1 1 5E8EB5AF
+L microsynth-rescue:SW_DPTT_SELECTOR-Switch SW9
+U 2 1 5E96003B
 P 2550 3700
-AR Path="/5E8EB5AF" Ref="SW9-TRIGGER1"  Part="1"
-AR Path="/5E8C1704/5E8EB5AF" Ref="SW9-TRIGGER1"  Part="1"
-F 0 "SW9-TRIGGER1" H 2744 3874 50  0000 L CNN
-F 1 "SW_DPTT_SELECTOR" H 2744 3783 50  0000 L CNN
+F 0 "SW9" H 2750 3850 50  0000 L CNN
+F 1 "SW_DPTT_SELECTOR-Switch" H 2750 3750 50  0000 L CNN
 F 2 "Buttons_Switches_ThroughHole:DP3T_Toggle" H 2550 3700 50  0001 C CNN
 F 3 "" H 2550 3700 50  0001 C CNN
-F 4 "TRIGGER" H 2744 3692 50  0000 L CNN "Label"
-	1    2550 3700
-	-1   0    0    1
-$EndComp
+	2    2550 3700
+	1    0    0    -1
+$EndComp
+$Comp
+L Device:R R27
+U 1 1 5E9A7E20
+P 4250 1300
+F 0 "R27" V 4000 1300 50  0000 C CNN
+F 1 "1k2" V 4100 1300 50  0000 C CNN
+F 2 "Resistor_THT:R_Axial_DIN0207_L6.3mm_D2.5mm_P10.16mm_Horizontal" V 4180 1300 50  0001 C CNN
+F 3 "~" H 4250 1300 50  0001 C CNN
+	1    4250 1300
+	0    1    1    0
+$EndComp
+Wire Wire Line
+	4400 1300 4700 1300
+$Comp
+L Device:R R2
+U 1 1 5E9E2792
+P 1800 1300
+F 0 "R2" V 1550 1300 50  0000 C CNN
+F 1 "680" V 1650 1300 50  0000 C CNN
+F 2 "Resistor_THT:R_Axial_DIN0207_L6.3mm_D2.5mm_P10.16mm_Horizontal" V 1730 1300 50  0001 C CNN
+F 3 "~" H 1800 1300 50  0001 C CNN
+	1    1800 1300
+	0    1    1    0
+$EndComp
+Wire Wire Line
+	1950 1300 3000 1300
 $EndSCHEMATC
