File: microsynth/Keyboard.sch (KiCad schematic (older format))
At the start: 55 parts, among them J6 Conn_01x02_Male, J7 Conn_01x02_Male, Q1 BC182, Q2 BC182L, SW1-DRIFT1 SW_DPTT_SELECTOR, SW9 SW_DPTT_SELECTOR-Switch, U1 TL074, U2 TL072, U3 4011, U4 4016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

Commit message: Laying out pcb
Parts:
- removed J6, J7: Conn_01x02_Male, Connector_PinHeader_2.54mm:PinHeader_1x02_P2.54mm_Vertical, symbol Connector:Conn_01x02_Male
- removed U1, U5: TL074, Package_DIP:DIP-14_W7.62mm, symbol Amplifier_Operational:TL074
- added U1: RC4136, Package_DIP:DIP-14_W7.62mm_LongPads, symbol Amplifier_Operational:RC4136
- added unit 3 of U2
- added U5: LF347, Package_DIP:DIP-14_W7.62mm_LongPads, symbol Amplifier_Operational:LF347
- C7: symbol Device:C -> Device:C_Small
- Q1, Q2: symbol Device:Q_NPN_BCE -> Device:Q_NPN_ECB
- SW1-DRIFT1: value SW_DPTT_SELECTOR -> DRIFT
- SW9: value SW_DPTT_SELECTOR-Switch -> TRIGGER
- renumbered RV2-GLIDE1 to RV2, RV3-SCALE1 to RV3
Connections:
- net +VSW: now also U1.11 (V+), U2.8 (V+), U5.4 (V+)
- net -VSW: now also U1.7 (V-), U2.4 (V-), U5.11 (V-)
- net GND: now also Q1.3 (B), U2.3 (+), U1.5 (+); no longer Q1.1 (B), U2.2 (-)
- net KEYBOARD_LOW_END: now reaches R27.2
- net KEYBOARD_HIGH_END: now reaches R2.1
- net at C7.1, R152.1, R39.1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: now also Q2.3 (B), R38.1; no longer Q2.1 (B), RV3.2, RV3.3
- net at D1.2 (A), U2.6 (-), U2.7: now also Q2.1 (E); no longer Q2.3 (E)
- net at C6.1, R37.2, U2.5 (+): now also Q1.1 (E); no longer Q1.3 (E)
- net at C1.1, SW1-DRIFT1.2, SW1-DRIFT1.3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: now also U5.3 (+); no longer C4.1, R33.2
- net at U3.1, U4.13: now also U1.3
- net at R29.2, R30.1: now also U1.1 (-)
- net at R1.1, R2.2: now also U1.6 (-)
- net at R140.2, R141.2, R33.1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: now also U2.2 (-); no longer U2.3 (+)
- net at RV3.1: now also U6.2 (-), U6.6; no longer R38.1
- net at R27.1: now also U1.4
- net at D3.2 (A): now also U1.10
- net at D2.2 (A): now also U1.12
- net at R47.2: now also U1.14 (-)
- net at R48.2: now also U1.13 (+)
- net at R49.2: now also U1.8 (-)
- net at R50.2: now also U1.9 (+)
- net FROM_KEYBOARD_CONTACTS renamed KEYBOARD_BUS
- net TO_KEYBOARD_CONTACTS renamed TRIGGER_BUS
- net TRIGGER_BUS: now also U1.2 (+)
- new net: C4.1, R33.2, U5.1, U5.2 (-)
- new net: R38.2, RV3.2, RV3.3
Other:
- moved on the sheet: C7, R152, R38, R39, R40, RV3

Commit message: Laying out pcb ...
Parts:
- added J5: Conn_01x02_Male, Connector_PinHeader_2.54mm:PinHeader_1x02_P2.54mm_Vertical, symbol Connector:Conn_01x02_Male
Connections:
- net VOUT_TO_SEQ_SKT: now also J5.2 (Pin_2); no longer C5.1, RV2.3, U6.3 (+)
- new net: C5.1, J5.1 (Pin_1), RV2.3, U6.3 (+)
Changed lines of the file:
@@
 	8150 2350 8100 2350
-Wire Wire Line
-	7950 2200 7950 2150
-Wire Wire Line
-	7950 2150 8300 2150
-Wire Wire Line
-	8300 2150 8300 2350
 Wire Wire Line
 	8300 2350 8150 2350
 Connection ~ 8150 2350
-Wire Wire Line
-	8300 1850 8300 2150
-Connection ~ 8300 2150
 $Comp
 L power:+VSW #PWR0217
@@
 Wire Wire Line
 	8300 2400 8300 2350
-Connection ~ 8300 2350
 Wire Wire Line
 	8350 2600 8300 2600
@@
 Text GLabel 8000 1700 2    50   BiDi ~ 0
 TO_S14_LFO_MOD
-Text GLabel 8300 1850 0    50   BiDi ~ 0
+Text GLabel 7950 1850 2    50   BiDi ~ 0
 VOUT_TO_SEQ_SKT
 Text GLabel 4300 4150 0    50   BiDi ~ 0
@@
 	1450 1900 1300 1900
 Connection ~ 1300 1900
+$Comp
+L Connector:Conn_01x02_Male J5
+U 1 1 5E8F2B9E
+P 8150 1950
+F 0 "J5" V 8200 2000 50  0000 L CNN
+F 1 "Conn_01x02_Male" V 8300 2000 50  0000 L CNN
+F 2 "Connector_PinHeader_2.54mm:PinHeader_1x02_P2.54mm_Vertical" H 8150 1950 50  0001 C CNN
+F 3 "~" H 8150 1950 50  0001 C CNN
+	1    8150 1950
+	0    1    1    0
+$EndComp
+Wire Wire Line
+	7950 1850 7950 2150
+Wire Wire Line
+	7950 2150 8050 2150
+Connection ~ 7950 2150
+Wire Wire Line
+	7950 2150 7950 2200
+Wire Wire Line
+	8150 2150 8150 2350
 $EndSCHEMATC

Commit message: Layout...
Parts:
- SW1-DRIFT1: footprint Buttons_Switches_ThroughHole:DP3T_Toggle -> Buttons_Switches_ThroughHole:OS203013MT8QN1
Connections:
- net at C7.1, Q2.3 (B), R38.1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: no longer R152.1
- net at R140.2, R141.2, R33.1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: now also R152.1
Other:
- moved on the sheet: R140, R141, R152, R32, R35, R41
Changed lines of the file:
@@
 F 0 "SW1" H 5844 1083 50  0000 L CNN
 F 1 "DRIFT" H 5844 992 50  0000 L CNN
-F 2 "Buttons_Switches_ThroughHole:DP3T_Toggle" H 5650 1050 50  0001 C CNN
-F 3 "" H 5650 1050 50  0001 C CNN
+F 2 "Buttons_Switches_ThroughHole:OS203013MT8QN1" H 5650 1050 50  0001 C CNN
+F 3 "https://www.tme.eu/Document/aa2d40399ed88e2cc02320a01dfb97ce/OSseries.pdf" H 5650 1050 50  0001 C CNN
 F 4 "DRIFT" H 5844 901 50  0000 L CNN "Label"
 	1    5650 1050
@@
 L Device:R R32
 U 1 1 5E9262E1
-P 6250 1250
-F 0 "R32" V 6043 1250 50  0000 C CNN
-F 1 "10M" V 6134 1250 50  0000 C CNN
-F 2 "Resistor_THT:R_Axial_DIN0207_L6.3mm_D2.5mm_P10.16mm_Horizontal" V 6180 1250 50  0001 C CNN
-F 3 "~" H 6250 1250 50  0001 C CNN
-	1    6250 1250
+P 6150 1250
+F 0 "R32" V 5943 1250 50  0000 C CNN
+F 1 "10M" V 6034 1250 50  0000 C CNN
+F 2 "Resistor_THT:R_Axial_DIN0207_L6.3mm_D2.5mm_P10.16mm_Horizontal" V 6080 1250 50  0001 C CNN
+F 3 "~" H 6150 1250 50  0001 C CNN
+	1    6150 1250
 	0    1    -1   0
 $EndComp
 Wire Wire Line
-	6100 1250 5800 1250
+	6000 1250 5800 1250
 $Comp
 L power:-VSW #PWR0208
@@
 $EndComp
 Wire Wire Line
-	6750 1000 6650 1000
-Wire Wire Line
-	6500 1000 6500 1250
-Wire Wire Line
-	6500 1250 6400 1250
+	6350 1000 6350 1250
+Wire Wire Line
+	6350 1250 6300 1250
 $Comp
 L Device:R R35
 U 1 1 5E930BCA
-P 6650 1500
-F 0 "R35" H 6720 1546 50  0000 L CNN
-F 1 "180k" H 6720 1455 50  0000 L CNN
-F 2 "Resistor_THT:R_Axial_DIN0207_L6.3mm_D2.5mm_P10.16mm_Horizontal" V 6580 1500 50  0001 C CNN
-F 3 "~" H 6650 1500 50  0001 C CNN
-	1    6650 1500
+P 6550 1500
+F 0 "R35" H 6620 1546 50  0000 L CNN
+F 1 "180k" H 6620 1455 50  0000 L CNN
+F 2 "Resistor_THT:R_Axial_DIN0207_L6.3mm_D2.5mm_P10.16mm_Horizontal" V 6480 1500 50  0001 C CNN
+F 3 "~" H 6550 1500 50  0001 C CNN
+	1    6550 1500
 	1    0    0    -1
 $EndComp
@@
 	7000 2250 7000 2000
 Wire Wire Line
-	6650 1650 6650 1800
-Wire Wire Line
-	6650 1800 7000 1800
+	6550 1650 6550 1800
+Wire Wire Line
+	6550 1800 7000 1800
 Connection ~ 7000 1800
 Wire Wire Line
@@
 Wire Wire Line
 	6750 1150 6750 1000
-Connection ~ 6750 1000
-Wire Wire Line
-	6650 1350 6650 1000
-Connection ~ 6650 1000
-Wire Wire Line
-	6650 1000 6500 1000
+Wire Wire Line
+	6550 1350 6550 1000
 Wire Wire Line
 	7000 1300 7000 1350
@@
 L power:+VSW #PWR0209
 U 1 1 5E93EA0A
-P 7450 800
-F 0 "#PWR0209" H 7450 650 50  0001 C CNN
-F 1 "+VSW" H 7465 973 50  0000 C CNN
-F 2 "" H 7450 800 50  0001 C CNN
-F 3 "" H 7450 800 50  0001 C CNN
-	1    7450 800
-	1    0    0    -1
-$EndComp
-Wire Wire Line
-	7450 800  7450 1150
+P 7450 1000
+F 0 "#PWR0209" H 7450 850 50  0001 C CNN
+F 1 "+VSW" H 7465 1173 50  0000 C CNN
+F 2 "" H 7450 1000 50  0001 C CNN
+F 3 "" H 7450 1000 50  0001 C CNN
+	1    7450 1000
+	1    0    0    -1
+$EndComp
+Wire Wire Line
+	7450 1000 7450 1150
 Wire Wire Line
 	7450 1150 7150 1150
@@
 L Device:R R140
 U 1 1 5E940A1E
-P 7700 1350
-F 0 "R140" V 7493 1350 50  0000 C CNN
-F 1 "10K" V 7584 1350 50  0000 C CNN
-F 2 "Resistor_THT:R_Axial_DIN0207_L6.3mm_D2.5mm_P10.16mm_Horizontal" V 7630 1350 50  0001 C CNN
-F 3 "~" H 7700 1350 50  0001 C CNN
-	1    7700 1350
+P 7950 1350
+F 0 "R140" V 7743 1350 50  0000 C CNN
+F 1 "10K" V 7834 1350 50  0000 C CNN
+F 2 "Resistor_THT:R_Axial_DIN0207_L6.3mm_D2.5mm_P10.16mm_Horizontal" V 7880 1350 50  0001 C CNN
+F 3 "~" H 7950 1350 50  0001 C CNN
+	1    7950 1350
 	0    1    1    0
 $EndComp
@@
 L Device:R R141
 U 1 1 5E941296
-P 7700 1700
-F 0 "R141" V 7493 1700 50  0000 C CNN
-F 1 "10K" V 7584 1700 50  0000 C CNN
-F 2 "Resistor_THT:R_Axial_DIN0207_L6.3mm_D2.5mm_P10.16mm_Horizontal" V 7630 1700 50  0001 C CNN
-F 3 "~" H 7700 1700 50  0001 C CNN
-	1    7700 1700
-	0    1    1    0
-$EndComp
-Wire Wire Line
-	7550 1700 7450 1700
+P 7950 1700
+F 0 "R141" V 7743 1700 50  0000 C CNN
+F 1 "10K" V 7834 1700 50  0000 C CNN
+F 2 "Resistor_THT:R_Axial_DIN0207_L6.3mm_D2.5mm_P10.16mm_Horizontal" V 7880 1700 50  0001 C CNN
+F 3 "~" H 7950 1700 50  0001 C CNN
+	1    7950 1700
+	0    1    1    0
+$EndComp
+Wire Wire Line
+	7800 1700 7650 1700
 Connection ~ 7000 1700
 Wire Wire Line
 	7000 1700 7000 1650
 Wire Wire Line
-	7450 1700 7450 1350
-Wire Wire Line
-	7450 1350 7550 1350
-Connection ~ 7450 1700
-Wire Wire Line
-	7450 1700 7000 1700
-Wire Wire Line
-	8000 1700 7850 1700
-Wire Wire Line
-	7950 1350 7850 1350
+	7650 1700 7650 1350
+Wire Wire Line
+	7650 1350 7800 1350
+Connection ~ 7650 1700
+Wire Wire Line
+	7650 1700 7000 1700
+Wire Wire Line
+	8200 1700 8100 1700
+Wire Wire Line
+	8200 1350 8100 1350
 $Comp
 L Device:R R34
@@
 L Device:R R152
 U 1 1 5E98598E
-P 9100 3200
-F 0 "R152" V 8893 3200 50  0000 C CNN
-F 1 "56k" V 8984 3200 50  0000 C CNN
-F 2 "Resistor_THT:R_Axial_DIN0207_L6.3mm_D2.5mm_P10.16mm_Horizontal" V 9030 3200 50  0001 C CNN
-F 3 "~" H 9100 3200 50  0001 C CNN
-	1    9100 3200
-	0    1    1    0
+P 7950 1000
+F 0 "R152" V 7743 1000 50  0000 C CNN
+F 1 "56k" V 7834 1000 50  0000 C CNN
+F 2 "Resistor_THT:R_Axial_DIN0207_L6.3mm_D2.5mm_P10.16mm_Horizontal" V 7880 1000 50  0001 C CNN
+F 3 "~" H 7950 1000 50  0001 C CNN
+	1    7950 1000
+	0    -1   1    0
 $EndComp
 $Comp
 L Device:R R41
 U 1 1 5E9860CB
-P 9100 3550
-F 0 "R41" V 8893 3550 50  0000 C CNN
-F 1 "39k" V 8984 3550 50  0000 C CNN
-F 2 "Resistor_THT:R_Axial_DIN0207_L6.3mm_D2.5mm_P10.16mm_Horizontal" V 9030 3550 50  0001 C CNN
-F 3 "~" H 9100 3550 50  0001 C CNN
-	1    9100 3550
-	0    1    1    0
-$EndComp
-Wire Wire Line
-	9250 3550 9450 3550
-Wire Wire Line
-	9450 3550 9450 3200
-Wire Wire Line
-	9450 3200 9250 3200
-Wire Wire Line
-	9450 3550 10400 3550
-Wire Wire Line
-	10400 3550 10400 2500
-Connection ~ 9450 3550
+P 9550 3600
+F 0 "R41" V 9343 3600 50  0000 C CNN
+F 1 "39k" V 9434 3600 50  0000 C CNN
+F 2 "Resistor_THT:R_Axial_DIN0207_L6.3mm_D2.5mm_P10.16mm_Horizontal" V 9480 3600 50  0001 C CNN
+F 3 "~" H 9550 3600 50  0001 C CNN
+	1    9550 3600
+	0    1    1    0
+$EndComp
+Wire Wire Line
+	7650 1350 7650 1000
+Wire Wire Line
+	7650 1000 7800 1000
+Wire Wire Line
+	10400 3600 10400 2500
 Connection ~ 10400 2500
 Wire Wire Line
-	8900 3200 8950 3200
-Wire Wire Line
-	8950 3550 8850 3550
+	8200 1000 8100 1000
+Wire Wire Line
+	9400 3600 9250 3600
 Wire Wire Line
 	6400 2700 6400 2600
@@
 Wire Wire Line
 	10700 2700 10700 3050
-Text GLabel 8850 3550 0    50   BiDi ~ 0
+Text GLabel 9250 3600 0    50   BiDi ~ 0
 TO_R41
-Text GLabel 7950 1350 2    50   BiDi ~ 0
+Text GLabel 8200 1350 2    50   BiDi ~ 0
 TO_S13_THUMBWEEL_MOD
-Text GLabel 8000 1700 2    50   BiDi ~ 0
+Text GLabel 8200 1700 2    50   BiDi ~ 0
 TO_S14_LFO_MOD
 Text GLabel 7950 1850 2    50   BiDi ~ 0
@@
 Text GLabel 3700 2800 2    50   BiDi ~ 0
 TRIG_OUT_TO_SEQ_SKT
-Text GLabel 8900 3200 0    50   BiDi ~ 0
+Text GLabel 8200 1000 2    50   BiDi ~ 0
 VIN_TO_SEQ_SKT
 Wire Wire Line
@@
 Wire Wire Line
 	8150 2150 8150 2350
+$Comp
+L power:-VSW #PWR0228
+U 1 1 5E98AA20
+P 6350 1000
+F 0 "#PWR0228" H 6350 1100 50  0001 C CNN
+F 1 "-VSW" H 6365 1173 50  0000 C CNN
+F 2 "" H 6350 1000 50  0001 C CNN
+F 3 "" H 6350 1000 50  0001 C CNN
+	1    6350 1000
+	1    0    0    -1
+$EndComp
+$Comp
+L power:-VSW #PWR0229
+U 1 1 5E98AE00
+P 6550 1000
+F 0 "#PWR0229" H 6550 1100 50  0001 C CNN
+F 1 "-VSW" H 6565 1173 50  0000 C CNN
+F 2 "" H 6550 1000 50  0001 C CNN
+F 3 "" H 6550 1000 50  0001 C CNN
+	1    6550 1000
+	1    0    0    -1
+$EndComp
+Connection ~ 7650 1350
+Wire Wire Line
+	9700 3600 10400 3600
 $EndSCHEMATC

Commit message: Layout...
Parts:
- SW1-DRIFT1: footprint Buttons_Switches_ThroughHole:OS203013MT8QN1 -> Buttons_Switches_ThroughHole:L203011MS02Q
Changed lines of the file:
@@
 F 0 "SW1" H 5844 1083 50  0000 L CNN
 F 1 "DRIFT" H 5844 992 50  0000 L CNN
-F 2 "Buttons_Switches_ThroughHole:OS203013MT8QN1" H 5650 1050 50  0001 C CNN
+F 2 "Buttons_Switches_ThroughHole:L203011MS02Q" H 5650 1050 50  0001 C CNN
 F 3 "https://www.tme.eu/Document/aa2d40399ed88e2cc02320a01dfb97ce/OSseries.pdf" H 5650 1050 50  0001 C CNN
 F 4 "DRIFT" H 5844 901 50  0000 L CNN "Label"
