File: microsynth/VCO1.sch (KiCad schematic (older format))
At the start: 24 parts, among them IC11 LM741, IC12 LM741, IC5 TL074, SW22 SW_SPST, U13 LM741, U14 4016

Commit message: Footprints
Parts:
- U5: renamed from IC5; footprint (none) -> Package_DIP:DIP-14_W7.62mm
- renumbered IC11 to U11, IC12 to U12
Other:
- moved on the sheet: C15, RV13, U5E
Changed lines of the file:
@@
 $EndDescr
 $Comp
-L Amplifier_Operational:LM741 IC11
+L Amplifier_Operational:LM741 U11
 U 1 1 5E222F28
 P 2450 1800
-F 0 "IC11" H 2794 1754 50  0000 L CNN
+F 0 "U11" H 2794 1754 50  0000 L CNN
 F 1 "LM741" H 2794 1845 50  0000 L CNN
 F 2 "" H 2500 1850 50  0001 C CNN
@@
 $EndComp
 $Comp
-L Amplifier_Operational:LM741 IC12
+L Amplifier_Operational:LM741 U12
 U 1 1 5E2243B9
 P 4000 1800
-F 0 "IC12" H 4344 1754 50  0000 L CNN
+F 0 "U12" H 4344 1754 50  0000 L CNN
 F 1 "LM741" H 4344 1845 50  0000 L CNN
 F 2 "" H 4050 1850 50  0001 C CNN
@@
 $EndComp
 $Comp
-L Amplifier_Operational:TL074 IC5
+L Amplifier_Operational:TL074 U5
 U 4 1 5E22A998
 P 3150 1900
-F 0 "IC5" H 3150 1533 50  0000 C CNN
+F 0 "U5" H 3150 1533 50  0000 C CNN
 F 1 "TL074" H 3150 1624 50  0000 C CNN
-F 2 "" H 3100 2000 50  0001 C CNN
+F 2 "Package_DIP:DIP-14_W7.62mm" H 3100 2000 50  0001 C CNN
 F 3 "http://www.ti.com/lit/ds/symlink/tl071.pdf" H 3200 2100 50  0001 C CNN
 	4    3150 1900
@@
 $EndComp
 $Comp
-L Amplifier_Operational:TL074 IC5
+L Amplifier_Operational:TL074 U5
 U 5 1 5E22BD33
-P 7650 1300
-F 0 "IC5" H 7608 1346 50  0000 L CNN
-F 1 "TL074" H 7608 1255 50  0000 L CNN
-F 2 "" H 7600 1400 50  0001 C CNN
-F 3 "http://www.ti.com/lit/ds/symlink/tl071.pdf" H 7700 1500 50  0001 C CNN
-	5    7650 1300
-	1    0    0    -1
-$EndComp
-Wire Wire Line
-	2750 1800 2800 1800
+P 6850 2950
+F 0 "U5" H 6808 2996 50  0000 L CNN
+F 1 "TL074" H 6808 2905 50  0000 L CNN
+F 2 "Package_DIP:DIP-14_W7.62mm" H 6800 3050 50  0001 C CNN
+F 3 "http://www.ti.com/lit/ds/symlink/tl071.pdf" H 6900 3150 50  0001 C CNN
+	5    6850 2950
+	1    0    0    -1
+$EndComp
 $Comp
 L Device:R R73
@@
 L Device:R_POT RV13
 U 1 1 5E254AE8
-P 2650 1250
-F 0 "RV13" V 2535 1250 50  0000 C CNN
-F 1 "10k" V 2444 1250 50  0000 C CNN
-F 2 "" H 2650 1250 50  0001 C CNN
-F 3 "~" H 2650 1250 50  0001 C CNN
-	1    2650 1250
+P 2650 950
+F 0 "RV13" V 2535 950 50  0000 C CNN
+F 1 "10k" V 2444 950 50  0000 C CNN
+F 2 "" H 2650 950 50  0001 C CNN
+F 3 "~" H 2650 950 50  0001 C CNN
+	1    2650 950
 	0    -1   -1   0
 $EndComp
@@
 L power:-VSW #PWR0143
 U 1 1 5E259E1E
-P 2650 1100
-F 0 "#PWR0143" H 2650 1200 50  0001 C CNN
-F 1 "-VSW" H 2665 1273 50  0000 C CNN
-F 2 "" H 2650 1100 50  0001 C CNN
-F 3 "" H 2650 1100 50  0001 C CNN
-	1    2650 1100
+P 2650 800
+F 0 "#PWR0143" H 2650 900 50  0001 C CNN
+F 1 "-VSW" H 2665 973 50  0000 C CNN
+F 2 "" H 2650 800 50  0001 C CNN
+F 3 "" H 2650 800 50  0001 C CNN
+	1    2650 800
 	1    0    0    -1
 $EndComp
@@
 Wire Wire Line
 	1350 3450 2450 3450
-Wire Wire Line
-	2450 1500 2450 1250
-Wire Wire Line
-	2450 1250 2500 1250
-Wire Wire Line
-	2800 1250 2900 1250
-Wire Wire Line
-	2900 1250 2900 1500
 $Comp
 L Device:C C15
 U 1 1 5E27DCDC
-P 2450 1400
-F 0 "C15" V 2198 1400 50  0000 C CNN
-F 1 "10n" V 2289 1400 50  0000 C CNN
-F 2 "" H 2488 1250 50  0001 C CNN
-F 3 "~" H 2450 1400 50  0001 C CNN
-	1    2450 1400
-	0    1    1    0
-$EndComp
-Wire Wire Line
-	2600 1400 2800 1800
-Connection ~ 2800 1800
-Wire Wire Line
-	2800 1800 2850 1800
+P 2550 1400
+F 0 "C15" V 2298 1400 50  0000 C CNN
+F 1 "10n" V 2389 1400 50  0000 C CNN
+F 2 "" H 2588 1250 50  0001 C CNN
+F 3 "~" H 2550 1400 50  0001 C CNN
+	1    2550 1400
+	0    1    1    0
+$EndComp
 Wire Wire Line
 	2150 1700 2150 1400
 Wire Wire Line
-	2150 1400 2300 1400
+	2150 1400 2400 1400
 Connection ~ 2150 1700
 Wire Wire Line
-	2600 1400 3700 1400
+	2700 1400 2800 1400
 Wire Wire Line
 	3700 1400 4450 1400
@@
 L power:-VSW #PWR0149
 U 1 1 5E2BC497
-P 7550 1600
-F 0 "#PWR0149" H 7550 1700 50  0001 C CNN
-F 1 "-VSW" H 7565 1773 50  0000 C CNN
-F 2 "" H 7550 1600 50  0001 C CNN
-F 3 "" H 7550 1600 50  0001 C CNN
-	1    7550 1600
+P 6750 3250
+F 0 "#PWR0149" H 6750 3350 50  0001 C CNN
+F 1 "-VSW" H 6765 3423 50  0000 C CNN
+F 2 "" H 6750 3250 50  0001 C CNN
+F 3 "" H 6750 3250 50  0001 C CNN
+	1    6750 3250
 	-1   0    0    1
 $EndComp
@@
 L power:+VSW #PWR0150
 U 1 1 5E2BCF5A
-P 7550 1000
-F 0 "#PWR0150" H 7550 850 50  0001 C CNN
-F 1 "+VSW" H 7565 1173 50  0000 C CNN
-F 2 "" H 7550 1000 50  0001 C CNN
-F 3 "" H 7550 1000 50  0001 C CNN
-	1    7550 1000
+P 6750 2650
+F 0 "#PWR0150" H 6750 2500 50  0001 C CNN
+F 1 "+VSW" H 6765 2823 50  0000 C CNN
+F 2 "" H 6750 2650 50  0001 C CNN
+F 3 "" H 6750 2650 50  0001 C CNN
+	1    6750 2650
 	1    0    0    -1
 $EndComp
@@
 Wire Wire Line
 	2750 2350 2750 2000
-Connection ~ 2600 1400
 Wire Wire Line
 	850  1250 850  1700
@@
 	-1   0    0    1
 $EndComp
+Wire Wire Line
+	2750 1800 2800 1800
+Wire Wire Line
+	2800 1800 2800 1400
+Connection ~ 2800 1800
+Wire Wire Line
+	2800 1800 2850 1800
+Connection ~ 2800 1400
+Wire Wire Line
+	2800 1400 3700 1400
+Wire Wire Line
+	2900 950  2800 950
+Wire Wire Line
+	2900 950  2900 1500
+Wire Wire Line
+	2450 950  2500 950
+Wire Wire Line
+	2450 950  2450 1500
 $EndSCHEMATC

Commit message: Footprints 2
Parts:
- C15, C16, C17: footprint (none) -> Capacitor_THT:C_Disc_D5.0mm_W2.5mm_P5.00mm
- U11, U12, U13: footprint (none) -> Package_DIP:DIP-8_W7.62mm_LongPads
- U14: footprint (none) -> Package_DIP:DIP-14_W7.62mm_LongPads
Changed lines of the file:
@@
 F 0 "U11" H 2794 1754 50  0000 L CNN
 F 1 "LM741" H 2794 1845 50  0000 L CNN
-F 2 "" H 2500 1850 50  0001 C CNN
+F 2 "Package_DIP:DIP-8_W7.62mm_LongPads" H 2500 1850 50  0001 C CNN
 F 3 "http://www.ti.com/lit/ds/symlink/lm741.pdf" H 2600 1950 50  0001 C CNN
 	1    2450 1800
@@
 F 0 "U12" H 4344 1754 50  0000 L CNN
 F 1 "LM741" H 4344 1845 50  0000 L CNN
-F 2 "" H 4050 1850 50  0001 C CNN
+F 2 "Package_DIP:DIP-8_W7.62mm_LongPads" H 4050 1850 50  0001 C CNN
 F 3 "http://www.ti.com/lit/ds/symlink/lm741.pdf" H 4150 1950 50  0001 C CNN
 	1    4000 1800
@@
 F 0 "U13" H 3244 4204 50  0000 L CNN
 F 1 "LM741" H 3244 4295 50  0000 L CNN
-F 2 "" H 2950 4300 50  0001 C CNN
+F 2 "Package_DIP:DIP-8_W7.62mm_LongPads" H 2950 4300 50  0001 C CNN
 F 3 "http://www.ti.com/lit/ds/symlink/lm741.pdf" H 3050 4400 50  0001 C CNN
 	1    2900 4250
@@
 F 0 "C16" V 1598 3150 50  0000 C CNN
 F 1 "15n" V 1689 3150 50  0000 C CNN
-F 2 "" H 1888 3000 50  0001 C CNN
+F 2 "Capacitor_THT:C_Disc_D5.0mm_W2.5mm_P5.00mm" H 1888 3000 50  0001 C CNN
 F 3 "~" H 1850 3150 50  0001 C CNN
 	1    1850 3150
@@
 F 0 "C17" V 2698 3900 50  0000 C CNN
 F 1 "10n" V 2789 3900 50  0000 C CNN
-F 2 "" H 2988 3750 50  0001 C CNN
+F 2 "Capacitor_THT:C_Disc_D5.0mm_W2.5mm_P5.00mm" H 2988 3750 50  0001 C CNN
 F 3 "~" H 2950 3900 50  0001 C CNN
 	1    2950 3900
@@
 F 0 "C15" V 2298 1400 50  0000 C CNN
 F 1 "10n" V 2389 1400 50  0000 C CNN
-F 2 "" H 2588 1250 50  0001 C CNN
+F 2 "Capacitor_THT:C_Disc_D5.0mm_W2.5mm_P5.00mm" H 2588 1250 50  0001 C CNN
 F 3 "~" H 2550 1400 50  0001 C CNN
 	1    2550 1400
@@
 F 0 "U14" V 1554 2222 50  0000 R CNN
 F 1 "4016" V 1645 2222 50  0000 R CNN
-F 2 "" H 1600 2350 50  0001 C CNN
+F 2 "Package_DIP:DIP-14_W7.62mm_LongPads" H 1600 2350 50  0001 C CNN
 F 3 "http://www.ti.com/lit/ds/symlink/cd4016b.pdf" H 1600 2350 50  0001 C CNN
 	2    1600 2350
@@
 F 0 "U14" H 3150 3377 50  0000 C CNN
 F 1 "4016" H 3150 3286 50  0000 C CNN
-F 2 "" H 3150 3550 50  0001 C CNN
+F 2 "Package_DIP:DIP-14_W7.62mm_LongPads" H 3150 3550 50  0001 C CNN
 F 3 "http://www.ti.com/lit/ds/symlink/cd4016b.pdf" H 3150 3550 50  0001 C CNN
 	3    3150 3550
@@
 F 0 "U14" H 7630 2946 50  0000 L CNN
 F 1 "4016" H 7630 2855 50  0000 L CNN
-F 2 "" H 7400 2900 50  0001 C CNN
+F 2 "Package_DIP:DIP-14_W7.62mm_LongPads" H 7400 2900 50  0001 C CNN
 F 3 "http://www.ti.com/lit/ds/symlink/cd4016b.pdf" H 7400 2900 50  0001 C CNN
 	5    7400 2900

Commit message: Hacking together the footprints
Parts:
- RV13, RV15: footprint (none) -> Potentiometers:Potentiometer_Trimmer_Bourns_PV36W
- RV14: value 100k -> 100kLIN; footprint (none) -> 4ms_Potentiometer:Pot_16mm_NoDet_RV16AF-4A
- SW22: footprint (none) -> 4ms:SPDT_KIT
Changed lines of the file:
@@
 P 4200 2750
 F 0 "RV14" H 4130 2659 50  0000 R CNN
-F 1 "100k" H 4130 2750 50  0000 R CNN
-F 2 "" H 4200 2750 50  0001 C CNN
+F 1 "100kLIN" H 4130 2750 50  0000 R CNN
+F 2 "4ms_Potentiometer:Pot_16mm_NoDet_RV16AF-4A" H 4200 2750 50  0001 C CNN
 F 3 "~" H 4200 2750 50  0001 C CNN
 F 4 "VCO1 PWM" H 4130 2841 50  0000 R CNN "Label"
@@
 F 0 "RV13" V 2535 950 50  0000 C CNN
 F 1 "10k" V 2444 950 50  0000 C CNN
-F 2 "" H 2650 950 50  0001 C CNN
+F 2 "Potentiometers:Potentiometer_Trimmer_Bourns_PV36W" H 2650 950 50  0001 C CNN
 F 3 "~" H 2650 950 50  0001 C CNN
 	1    2650 950
@@
 F 0 "RV15" H 1130 3496 50  0000 R CNN
 F 1 "100k" H 1130 3405 50  0000 R CNN
-F 2 "" H 1200 3450 50  0001 C CNN
+F 2 "Potentiometers:Potentiometer_Trimmer_Bourns_PV36W" H 1200 3450 50  0001 C CNN
 F 3 "~" H 1200 3450 50  0001 C CNN
 	1    1200 3450
@@
 F 0 "SW22" V 1141 1162 50  0000 R CNN
 F 1 "SW_SPST" V 1050 1162 50  0000 R CNN
-F 2 "" H 1050 1250 50  0001 C CNN
+F 2 "4ms:SPDT_KIT" H 1050 1250 50  0001 C CNN
 F 3 "~" H 1050 1250 50  0001 C CNN
 F 4 "VCO1 On/Off" V 959 1162 50  0000 R CNN "Label"

Commit message: Laying out pcb
Parts:
- removed U5: TL074, Package_DIP:DIP-14_W7.62mm, symbol Amplifier_Operational:TL074
- added U5: LF347, Package_DIP:DIP-14_W7.62mm_LongPads, symbol Amplifier_Operational:LF347
Connections:
- net IC22_PIN_3: now also U5.14
- net VCO1_SAW1: now also U5.13 (-)
- net at R74.1, R75.1: now also U5.12 (+)
Changed lines of the file:
@@
 U 1 1 5E222F28
 P 2450 1800
-F 0 "U11" H 2794 1754 50  0000 L CNN
-F 1 "LM741" H 2794 1845 50  0000 L CNN
+F 0 "U11" H 2350 1800 50  0000 L CNN
+F 1 "LM741" H 2450 1950 50  0000 L CNN
 F 2 "Package_DIP:DIP-8_W7.62mm_LongPads" H 2500 1850 50  0001 C CNN
 F 3 "http://www.ti.com/lit/ds/symlink/lm741.pdf" H 2600 1950 50  0001 C CNN
@@
 U 1 1 5E2243B9
 P 4000 1800
-F 0 "U12" H 4344 1754 50  0000 L CNN
-F 1 "LM741" H 4344 1845 50  0000 L CNN
+F 0 "U12" H 3900 1800 50  0000 L CNN
+F 1 "LM741" H 3950 2000 50  0000 L CNN
 F 2 "Package_DIP:DIP-8_W7.62mm_LongPads" H 4050 1850 50  0001 C CNN
 F 3 "http://www.ti.com/lit/ds/symlink/lm741.pdf" H 4150 1950 50  0001 C CNN
@@
 	1    2900 4250
 	1    0    0    1
-$EndComp
-$Comp
-L Amplifier_Operational:TL074 U5
-U 4 1 5E22A998
-P 3150 1900
-F 0 "U5" H 3150 1533 50  0000 C CNN
-F 1 "TL074" H 3150 1624 50  0000 C CNN
-F 2 "Package_DIP:DIP-14_W7.62mm" H 3100 2000 50  0001 C CNN
-F 3 "http://www.ti.com/lit/ds/symlink/tl071.pdf" H 3200 2100 50  0001 C CNN
-	4    3150 1900
-	1    0    0    1
-$EndComp
-$Comp
-L Amplifier_Operational:TL074 U5
-U 5 1 5E22BD33
-P 6850 2950
-F 0 "U5" H 6808 2996 50  0000 L CNN
-F 1 "TL074" H 6808 2905 50  0000 L CNN
-F 2 "Package_DIP:DIP-14_W7.62mm" H 6800 3050 50  0001 C CNN
-F 3 "http://www.ti.com/lit/ds/symlink/tl071.pdf" H 6900 3150 50  0001 C CNN
-	5    6850 2950
-	1    0    0    -1
 $EndComp
 $Comp
@@
 	3700 1400 4450 1400
 Connection ~ 3700 1400
-$Comp
-L power:-VSW #PWR0149
-U 1 1 5E2BC497
-P 6750 3250
-F 0 "#PWR0149" H 6750 3350 50  0001 C CNN
-F 1 "-VSW" H 6765 3423 50  0000 C CNN
-F 2 "" H 6750 3250 50  0001 C CNN
-F 3 "" H 6750 3250 50  0001 C CNN
-	1    6750 3250
-	-1   0    0    1
-$EndComp
-$Comp
-L power:+VSW #PWR0150
-U 1 1 5E2BCF5A
-P 6750 2650
-F 0 "#PWR0150" H 6750 2500 50  0001 C CNN
-F 1 "+VSW" H 6765 2823 50  0000 C CNN
-F 2 "" H 6750 2650 50  0001 C CNN
-F 3 "" H 6750 2650 50  0001 C CNN
-	1    6750 2650
-	1    0    0    -1
-$EndComp
 Wire Wire Line
 	2750 2400 2750 2350
@@
 Wire Wire Line
 	2450 950  2450 1500
+$Comp
+L Amplifier_Operational:LF347 U?
+U 4 1 5E920B31
+P 3150 1900
+AR Path="/5E8C1704/5E920B31" Ref="U?"  Part="4"
+AR Path="/5E222DC1/5E920B31" Ref="U5"  Part="4"
+F 0 "U5" H 3150 1500 50  0000 C CNN
+F 1 "LF347" H 3150 1600 50  0000 C CNN
+F 2 "Package_DIP:DIP-14_W7.62mm_LongPads" H 3100 2000 50  0001 C CNN
+F 3 "https://www.ti.com/lit/ds/symlink/lf147.pdf" H 3200 2100 50  0001 C CNN
+	4    3150 1900
+	1    0    0    1
+$EndComp
 $EndSCHEMATC

Commit message: Laying out pcb ...
Connections:
- net GND: now also RV15.1; no longer RV15.3
- net at C16.2: now also RV15.3; no longer RV15.1
Other:
- moved on the sheet: U13
Changed lines of the file:
@@
 L Amplifier_Operational:LM741 U13
 U 1 1 5E224C5D
-P 2900 4250
-F 0 "U13" H 3244 4204 50  0000 L CNN
-F 1 "LM741" H 3244 4295 50  0000 L CNN
-F 2 "Package_DIP:DIP-8_W7.62mm_LongPads" H 2950 4300 50  0001 C CNN
-F 3 "http://www.ti.com/lit/ds/symlink/lm741.pdf" H 3050 4400 50  0001 C CNN
-	1    2900 4250
+P 2900 4450
+F 0 "U13" H 3244 4404 50  0000 L CNN
+F 1 "LM741" H 3244 4495 50  0000 L CNN
+F 2 "Package_DIP:DIP-8_W7.62mm_LongPads" H 2950 4500 50  0001 C CNN
+F 3 "http://www.ti.com/lit/ds/symlink/lm741.pdf" H 3050 4600 50  0001 C CNN
+	1    2900 4450
 	1    0    0    1
 $EndComp
@@
 L power:+VSW #PWR0144
 U 1 1 5E25E987
-P 2800 4550
-F 0 "#PWR0144" H 2800 4400 50  0001 C CNN
-F 1 "+VSW" H 2815 4723 50  0000 C CNN
-F 2 "" H 2800 4550 50  0001 C CNN
-F 3 "" H 2800 4550 50  0001 C CNN
-	1    2800 4550
+P 2800 4750
+F 0 "#PWR0144" H 2800 4600 50  0001 C CNN
+F 1 "+VSW" H 2815 4923 50  0000 C CNN
+F 2 "" H 2800 4750 50  0001 C CNN
+F 3 "" H 2800 4750 50  0001 C CNN
+	1    2800 4750
 	-1   0    0    1
 $EndComp
@@
 L power:-VSW #PWR0145
 U 1 1 5E25EF82
-P 2800 3950
-F 0 "#PWR0145" H 2800 4050 50  0001 C CNN
-F 1 "-VSW" H 2815 4123 50  0000 C CNN
-F 2 "" H 2800 3950 50  0001 C CNN
-F 3 "" H 2800 3950 50  0001 C CNN
-	1    2800 3950
-	1    0    0    -1
-$EndComp
-NoConn ~ 2900 3950
-NoConn ~ 3000 3950
-Wire Wire Line
-	3200 4250 3450 4250
-Wire Wire Line
-	3450 4250 3450 3900
-Wire Wire Line
-	2450 4150 2600 4150
+P 2800 4150
+F 0 "#PWR0145" H 2800 4250 50  0001 C CNN
+F 1 "-VSW" H 2815 4323 50  0000 C CNN
+F 2 "" H 2800 4150 50  0001 C CNN
+F 3 "" H 2800 4150 50  0001 C CNN
+	1    2800 4150
+	1    0    0    -1
+$EndComp
+NoConn ~ 2900 4150
+NoConn ~ 3000 4150
+Wire Wire Line
+	3200 4450 3450 4450
 $Comp
 L Device:R_POT RV15
@@
 F 3 "~" H 1200 3450 50  0001 C CNN
 	1    1200 3450
-	1    0    0    -1
+	1    0    0    1
 $EndComp
 $Comp
@@
 L power:GND #PWR0148
 U 1 1 5E267D40
-P 2550 4700
-F 0 "#PWR0148" H 2550 4450 50  0001 C CNN
-F 1 "GND" H 2555 4527 50  0000 C CNN
-F 2 "" H 2550 4700 50  0001 C CNN
-F 3 "" H 2550 4700 50  0001 C CNN
-	1    2550 4700
-	1    0    0    -1
-$EndComp
-Wire Wire Line
-	2550 4700 2550 4350
+P 2550 4900
+F 0 "#PWR0148" H 2550 4650 50  0001 C CNN
+F 1 "GND" H 2555 4727 50  0000 C CNN
+F 2 "" H 2550 4900 50  0001 C CNN
+F 3 "" H 2550 4900 50  0001 C CNN
+	1    2550 4900
+	1    0    0    -1
+$EndComp
+Wire Wire Line
+	2550 4900 2550 4550
 $Comp
 L Device:R R76
@@
 Wire Wire Line
 	2000 4150 2450 4150
-Connection ~ 2450 4150
 Wire Wire Line
 	1700 4150 850  4150
@@
 	5250 3550 3450 3550
 Wire Wire Line
-	2550 4350 2600 4350
+	2550 4550 2600 4550
 Wire Wire Line
 	3700 1400 3700 1700
@@
 	1    0    0    1
 $EndComp
+Wire Wire Line
+	2450 4150 2450 4350
+Wire Wire Line
+	2450 4350 2600 4350
+Connection ~ 2450 4150
+Wire Wire Line
+	3450 3900 3450 4450
 $EndSCHEMATC

Commit message: Layout...
Connections:
- net KEYBOARD_OUTPUT: now also SW22.1 (A); no longer SW22.2 (B)
- net at R70.1, R72.2, R76.2: now also SW22.2 (B); no longer SW22.1 (A)
Changed lines of the file:
@@
 	850  1700 1100 1700
 Connection ~ 1100 1700
-$Comp
-L Switch:SW_SPST SW22
-U 1 1 5E26DDD4
-P 1050 1250
-F 0 "SW22" V 1141 1162 50  0000 R CNN
-F 1 "SW_SPST" V 1050 1162 50  0000 R CNN
-F 2 "4ms:SPDT_KIT" H 1050 1250 50  0001 C CNN
-F 3 "~" H 1050 1250 50  0001 C CNN
-F 4 "VCO1 On/Off" V 959 1162 50  0000 R CNN "Label"
-	1    1050 1250
-	1    0    0    -1
-$EndComp
 Wire Wire Line
 	1200 3300 1200 3150
@@
 Wire Wire Line
 	3450 3900 3450 4450
+$Comp
+L Switch:SW_SPST SW22
+U 1 1 5E26DDD4
+P 1050 1250
+F 0 "SW22" V 1141 1162 50  0000 R CNN
+F 1 "SW_SPST" V 1050 1162 50  0000 R CNN
+F 2 "4ms:SPDT_KIT" H 1050 1250 50  0001 C CNN
+F 3 "~" H 1050 1250 50  0001 C CNN
+F 4 "VCO1 On/Off" V 959 1162 50  0000 R CNN "Label"
+	1    1050 1250
+	-1   0    0    -1
+$EndComp
 $EndSCHEMATC

Commit message: Tidy up, name switches, proper footprints for all trimmers
Changed lines of the file:
@@
 P 2650 950
 F 0 "RV13" V 2535 950 50  0000 C CNN
-F 1 "10k" V 2444 950 50  0000 C CNN
+F 1 "10k" V 2800 850 50  0000 C CNN
 F 2 "Potentiometers:Potentiometer_Trimmer_Bourns_PV36W" H 2650 950 50  0001 C CNN
 F 3 "~" H 2650 950 50  0001 C CNN
