File: microsynth/VCA.sch (KiCad schematic (older format))
At the start: 32 parts, among them J1 AudioJack3, Q9 BC548, U21 CA3080, U23 LM380N

Commit message: Footprints 2
Parts:
- C26, C27, C28, C33: footprint (none) -> Capacitor_THT:C_Disc_D5.0mm_W2.5mm_P5.00mm
- C29, C30, C31, C32, C34: footprint (none) -> Capacitor_THT:CP_Radial_D10.0mm_P5.00mm
- J1: footprint (none) -> Connector_Audio:Jack_3.5mm_QingPu_WQP-PJ398SM_Vertical_CircularHoles
- Q9: footprint Package_TO_SOT_THT:TO-92_Inline -> Package_TO_SOT_THT:TO-92L_Inline_Wide
Changed lines of the file:
@@
 F 0 "C30" V 2555 950 50  0000 C CNN
 F 1 "4.7u" V 2464 950 50  0000 C CNN
-F 2 "" H 2338 800 50  0001 C CNN
+F 2 "Capacitor_THT:CP_Radial_D10.0mm_P5.00mm" H 2338 800 50  0001 C CNN
 F 3 "~" H 2300 950 50  0001 C CNN
 	1    2300 950
@@
 F 0 "C26" V 1048 2650 50  0000 C CNN
 F 1 "220n" V 1139 2650 50  0000 C CNN
-F 2 "" H 1338 2500 50  0001 C CNN
+F 2 "Capacitor_THT:C_Disc_D5.0mm_W2.5mm_P5.00mm" H 1338 2500 50  0001 C CNN
 F 3 "~" H 1300 2650 50  0001 C CNN
 	1    1300 2650
@@
 F 0 "C27" V 1552 3050 50  0000 C CNN
 F 1 "220n" V 1461 3050 50  0000 C CNN
-F 2 "" H 1338 2900 50  0001 C CNN
+F 2 "Capacitor_THT:C_Disc_D5.0mm_W2.5mm_P5.00mm" H 1338 2900 50  0001 C CNN
 F 3 "~" H 1300 3050 50  0001 C CNN
 	1    1300 3050
@@
 F 0 "C28" V 1552 3450 50  0000 C CNN
 F 1 "220n" V 1461 3450 50  0000 C CNN
-F 2 "" H 1338 3300 50  0001 C CNN
+F 2 "Capacitor_THT:C_Disc_D5.0mm_W2.5mm_P5.00mm" H 1338 3300 50  0001 C CNN
 F 3 "~" H 1300 3450 50  0001 C CNN
 	1    1300 3450
@@
 F 0 "Q9" H 4041 2596 50  0000 L CNN
 F 1 "BC548" H 4041 2505 50  0000 L CNN
-F 2 "Package_TO_SOT_THT:TO-92_Inline" H 4050 2475 50  0001 L CIN
+F 2 "Package_TO_SOT_THT:TO-92L_Inline_Wide" H 4050 2475 50  0001 L CIN
 F 3 "http://www.fairchildsemi.com/ds/BC/BC547.pdf" H 3850 2550 50  0001 L CNN
 	1    3850 2550
@@
 F 0 "C29" V 4855 2500 50  0000 C CNN
 F 1 "4.7u" V 4764 2500 50  0000 C CNN
-F 2 "" H 4638 2350 50  0001 C CNN
+F 2 "Capacitor_THT:CP_Radial_D10.0mm_P5.00mm" H 4638 2350 50  0001 C CNN
 F 3 "~" H 4600 2500 50  0001 C CNN
 	1    4600 2500
@@
 F 0 "C31" V 6245 1800 50  0000 C CNN
 F 1 "4.7u" V 6336 1800 50  0000 C CNN
-F 2 "" H 6538 1650 50  0001 C CNN
+F 2 "Capacitor_THT:CP_Radial_D10.0mm_P5.00mm" H 6538 1650 50  0001 C CNN
 F 3 "~" H 6500 1800 50  0001 C CNN
 	1    6500 1800
@@
 F 0 "C34" V 8705 1700 50  0000 C CNN
 F 1 "470u" V 8614 1700 50  0000 C CNN
-F 2 "" H 8488 1550 50  0001 C CNN
+F 2 "Capacitor_THT:CP_Radial_D10.0mm_P5.00mm" H 8488 1550 50  0001 C CNN
 F 3 "~" H 8450 1700 50  0001 C CNN
 	1    8450 1700
@@
 F 0 "C32" H 7868 2346 50  0000 L CNN
 F 1 "4.7u" H 7868 2255 50  0000 L CNN
-F 2 "" H 7788 2150 50  0001 C CNN
+F 2 "Capacitor_THT:CP_Radial_D10.0mm_P5.00mm" H 7788 2150 50  0001 C CNN
 F 3 "~" H 7750 2300 50  0001 C CNN
 	1    7750 2300
@@
 F 0 "C33" H 8165 2596 50  0000 L CNN
 F 1 "100n" H 8165 2505 50  0000 L CNN
-F 2 "" H 8088 2400 50  0001 C CNN
+F 2 "Capacitor_THT:C_Disc_D5.0mm_W2.5mm_P5.00mm" H 8088 2400 50  0001 C CNN
 F 3 "~" H 8050 2550 50  0001 C CNN
 	1    8050 2550
@@
 F 0 "J1" H 9220 2125 50  0000 R CNN
 F 1 "AudioJack3" H 9220 2034 50  0000 R CNN
-F 2 "" H 9500 2100 50  0001 C CNN
+F 2 "Connector_Audio:Jack_3.5mm_QingPu_WQP-PJ398SM_Vertical_CircularHoles" H 9500 2100 50  0001 C CNN
 F 3 "~" H 9500 2100 50  0001 C CNN
 	1    9500 2100

Commit message: Hacking together the footprints
Parts:
- J1: footprint Connector_Audio:Jack_3.5mm_QingPu_WQP-PJ398SM_Vertical_CircularHoles -> 4ms_Jack:EighthInch_Stereo_PJ366ST_ALT
- RV25: footprint (none) -> Potentiometers:Potentiometer_Trimmer_Bourns_PV36W
- RV26: value 10k -> 10kLOG; footprint (none) -> 4ms_Potentiometer:Pot_16mm_NoDet_RV16AF-4A
Changed lines of the file:
@@
 F 0 "RV25" H 3130 3254 50  0000 R CNN
 F 1 "100k" H 3130 3345 50  0000 R CNN
-F 2 "" H 3200 3300 50  0001 C CNN
+F 2 "Potentiometers:Potentiometer_Trimmer_Bourns_PV36W" H 3200 3300 50  0001 C CNN
 F 3 "~" H 3200 3300 50  0001 C CNN
 	1    3200 3300
@@
 P 5000 3300
 F 0 "RV26" H 4930 3346 50  0000 R CNN
-F 1 "10k" H 4930 3255 50  0000 R CNN
-F 2 "" H 5000 3300 50  0001 C CNN
+F 1 "10kLOG" H 4930 3255 50  0000 R CNN
+F 2 "4ms_Potentiometer:Pot_16mm_NoDet_RV16AF-4A" H 5000 3300 50  0001 C CNN
 F 3 "~" H 5000 3300 50  0001 C CNN
 	1    5000 3300
@@
 F 0 "J1" H 9220 2125 50  0000 R CNN
 F 1 "AudioJack3" H 9220 2034 50  0000 R CNN
-F 2 "Connector_Audio:Jack_3.5mm_QingPu_WQP-PJ398SM_Vertical_CircularHoles" H 9500 2100 50  0001 C CNN
+F 2 "4ms_Jack:EighthInch_Stereo_PJ366ST_ALT" H 9500 2100 50  0001 C CNN
 F 3 "~" H 9500 2100 50  0001 C CNN
 	1    9500 2100

Commit message: All components placed on PCB
Parts:
- added J8: AudioJack2, 4ms_Jack:EighthInch_Stereo_PJ366ST_ALT, symbol Connector:AudioJack2
- C29, C30, C31, C32, C34: footprint Capacitor_THT:CP_Radial_D10.0mm_P5.00mm -> Capacitor_THT:CP_Radial_D5.0mm_P2.50mm
Connections:
- net GND: now also J8.T
- net at C31.2, RV26.2: now also J8.S
Changed lines of the file:
@@
 F 0 "C30" V 2555 950 50  0000 C CNN
 F 1 "4.7u" V 2464 950 50  0000 C CNN
-F 2 "Capacitor_THT:CP_Radial_D10.0mm_P5.00mm" H 2338 800 50  0001 C CNN
+F 2 "Capacitor_THT:CP_Radial_D5.0mm_P2.50mm" H 2338 800 50  0001 C CNN
 F 3 "~" H 2300 950 50  0001 C CNN
 	1    2300 950
@@
 U 1 1 5E1BA63E
 P 2850 2550
-F 0 "U21" H 3194 2596 50  0000 L CNN
-F 1 "CA3080" H 3194 2505 50  0000 L CNN
+F 0 "U21" H 2650 2550 50  0000 L CNN
+F 1 "CA3080" H 2850 2350 50  0000 L CNN
 F 2 "Package_DIP:DIP-8_W7.62mm_LongPads" H 2850 2550 50  0001 C CNN
 F 3 "http://www.intersil.com/content/dam/Intersil/documents/ca30/ca3080-a.pdf" H 2850 2650 50  0001 C CNN
@@
 F 0 "C29" V 4855 2500 50  0000 C CNN
 F 1 "4.7u" V 4764 2500 50  0000 C CNN
-F 2 "Capacitor_THT:CP_Radial_D10.0mm_P5.00mm" H 4638 2350 50  0001 C CNN
+F 2 "Capacitor_THT:CP_Radial_D5.0mm_P2.50mm" H 4638 2350 50  0001 C CNN
 F 3 "~" H 4600 2500 50  0001 C CNN
 	1    4600 2500
@@
 F 0 "C31" V 6245 1800 50  0000 C CNN
 F 1 "4.7u" V 6336 1800 50  0000 C CNN
-F 2 "Capacitor_THT:CP_Radial_D10.0mm_P5.00mm" H 6538 1650 50  0001 C CNN
+F 2 "Capacitor_THT:CP_Radial_D5.0mm_P2.50mm" H 6538 1650 50  0001 C CNN
 F 3 "~" H 6500 1800 50  0001 C CNN
 	1    6500 1800
@@
 F 0 "C34" V 8705 1700 50  0000 C CNN
 F 1 "470u" V 8614 1700 50  0000 C CNN
-F 2 "Capacitor_THT:CP_Radial_D10.0mm_P5.00mm" H 8488 1550 50  0001 C CNN
+F 2 "Capacitor_THT:CP_Radial_D5.0mm_P2.50mm" H 8488 1550 50  0001 C CNN
 F 3 "~" H 8450 1700 50  0001 C CNN
 	1    8450 1700
@@
 F 0 "C32" H 7868 2346 50  0000 L CNN
 F 1 "4.7u" H 7868 2255 50  0000 L CNN
-F 2 "Capacitor_THT:CP_Radial_D10.0mm_P5.00mm" H 7788 2150 50  0001 C CNN
+F 2 "Capacitor_THT:CP_Radial_D5.0mm_P2.50mm" H 7788 2150 50  0001 C CNN
 F 3 "~" H 7750 2300 50  0001 C CNN
 	1    7750 2300
@@
 U 1 1 5E1E7AED
 P 7350 1700
-F 0 "U23" H 7694 1746 50  0000 L CNN
-F 1 "LM380N" H 7694 1655 50  0000 L CNN
+F 0 "U23" H 7300 1700 50  0000 L CNN
+F 1 "LM380N" H 7400 1550 50  0000 L CNN
 F 2 "Package_DIP:DIP-14_W7.62mm" H 7350 1700 50  0001 C CIN
 F 3 "http://www.ti.com/lit/ds/symlink/lm380.pdf" H 7350 1700 50  0001 C CNN
@@
 Wire Wire Line
 	2050 5300 2150 5300
+$Comp
+L Connector:AudioJack2 J?
+U 1 1 5EA25E4A
+P 5900 3400
+AR Path="/5E05EC3F/5EA25E4A" Ref="J?"  Part="1"
+AR Path="/5E1B03E8/5EA25E4A" Ref="J8"  Part="1"
+F 0 "J8" H 5720 3520 50  0000 R CNN
+F 1 "AudioJack2" H 5720 3429 50  0000 R CNN
+F 2 "4ms_Jack:EighthInch_Stereo_PJ366ST_ALT" H 5900 3400 50  0001 C CNN
+F 3 "~" H 5900 3400 50  0001 C CNN
+F 4 "TRIGGER OUT" H 5720 3338 50  0000 R CNN "Label"
+	1    5900 3400
+	-1   0    0    -1
+$EndComp
+$Comp
+L power:GND #PWR01
+U 1 1 5EA2727A
+P 5700 3400
+F 0 "#PWR01" H 5700 3150 50  0001 C CNN
+F 1 "GND" H 5705 3227 50  0000 C CNN
+F 2 "" H 5700 3400 50  0001 C CNN
+F 3 "" H 5700 3400 50  0001 C CNN
+	1    5700 3400
+	1    0    0    -1
+$EndComp
 $EndSCHEMATC

Commit message: Laying out pcb
Parts:
- RV26: Label (none) -> Volume
Changed lines of the file:
@@
 F 2 "4ms_Potentiometer:Pot_16mm_NoDet_RV16AF-4A" H 5000 3300 50  0001 C CNN
 F 3 "~" H 5000 3300 50  0001 C CNN
+F 4 "Volume" H 4800 3150 50  0000 C BNN "Label"
 	1    5000 3300
 	1    0    0    -1

Commit message: Laying out pcb ...
Connections:
- net GND: now also RV26.1; no longer RV26.3
- net at R139.2: now also RV26.3; no longer RV26.1
Changed lines of the file:
@@
 F 4 "Volume" H 4800 3150 50  0000 C BNN "Label"
 	1    5000 3300
-	1    0    0    -1
+	1    0    0    1
 $EndComp
 Wire Wire Line

Commit message: Layout...
Connections:
- net LFO_MOD renamed LFO_MOD_S17
Changed lines of the file:
@@
 VCO1_TRI
 Text GLabel 2000 950  0    50   BiDi ~ 0
-LFO_MOD
+LFO_MOD_S17
 Text GLabel 2000 1250 0    50   BiDi ~ 0
 ADSR
@@
 	1    0    0    -1
 $EndComp
-Text GLabel 2150 5300 2    50   BiDi ~ 0
-TO_VCA_C30
-Text GLabel 2050 5300 0    50   BiDi ~ 0
-LFO_MOD
-Wire Wire Line
-	2050 5300 2150 5300
 $Comp
 L Connector:AudioJack2 J?

Commit message: Layout...-3
Parts:
- J1: footprint 4ms_Jack:EighthInch_Stereo_PJ366ST_ALT -> Connector_PinHeader_2.54mm:PinHeader_1x03_P2.54mm_Vertical; symbol Connector:AudioJack3 -> Connector:Conn_01x03_Male; Label (none) -> STEREO OUT
- J8: footprint 4ms_Jack:EighthInch_Stereo_PJ366ST_ALT -> Connector_PinHeader_2.54mm:PinHeader_1x02_P2.54mm_Vertical; symbol Connector:AudioJack2 -> Connector:Conn_01x02_Male; Label TRIGGER OUT -> LINE OUT
- RV26: footprint 4ms_Potentiometer:Pot_16mm_NoDet_RV16AF-4A -> Connector_PinHeader_2.54mm:PinHeader_1x03_P2.54mm_Vertical
Connections:
- net GND: now also J1.3 (Pin_3), J8.2 (Pin_2); no longer J1.T, J8.T
- net at C31.2, RV26.2: now also J8.1 (Pin_1); no longer J8.S
- net at R146.1: now also J1.1 (Pin_1); no longer J1.S
- net at R145.2: now also J1.2 (Pin_2); no longer J1.R
- net HOLD_ON renamed TO_VCA_R136
Other:
- moved on the sheet: J8
Changed lines of the file:
@@
 	2850 1100 2850 1250
 $Comp
-L power:-VSW #PWR0125
+L power:-VSW #PWR?
 U 1 1 5E1BA11B
 P 3450 1100
-F 0 "#PWR0125" H 3450 1200 50  0001 C CNN
+F 0 "#PWR?" H 3450 1200 50  0001 C CNN
 F 1 "-VSW" H 3465 1273 50  0000 C CNN
 F 2 "" H 3450 1100 50  0001 C CNN
@@
 $EndComp
 $Comp
-L power:+VSW #PWR0126
+L power:+VSW #PWR?
 U 1 1 5E1BAC13
 P 2750 2250
-F 0 "#PWR0126" H 2750 2100 50  0001 C CNN
+F 0 "#PWR?" H 2750 2100 50  0001 C CNN
 F 1 "+VSW" H 2765 2423 50  0000 C CNN
 F 2 "" H 2750 2250 50  0001 C CNN
@@
 $EndComp
 $Comp
-L power:-VSW #PWR0127
+L power:-VSW #PWR?
 U 1 1 5E1BB094
 P 2750 2850
-F 0 "#PWR0127" H 2750 2950 50  0001 C CNN
+F 0 "#PWR?" H 2750 2950 50  0001 C CNN
 F 1 "-VSW" H 2765 3023 50  0000 C CNN
 F 2 "" H 2750 2850 50  0001 C CNN
@@
 	1950 3750 2300 3750
 $Comp
-L power:GND #PWR0128
+L power:GND #PWR?
 U 1 1 5E1D744F
 P 2300 3750
-F 0 "#PWR0128" H 2300 3500 50  0001 C CNN
+F 0 "#PWR?" H 2300 3500 50  0001 C CNN
 F 1 "GND" H 2305 3577 50  0000 C CNN
 F 2 "" H 2300 3750 50  0001 C CNN
@@
 $EndComp
 $Comp
-L power:+VSW #PWR0129
+L power:+VSW #PWR?
 U 1 1 5E1D84B3
 P 3950 2100
-F 0 "#PWR0129" H 3950 1950 50  0001 C CNN
+F 0 "#PWR?" H 3950 1950 50  0001 C CNN
 F 1 "+VSW" H 3965 2273 50  0000 C CNN
 F 2 "" H 3950 2100 50  0001 C CNN
@@
 	3950 2850 3950 2800
 $Comp
-L power:+VSW #PWR0130
+L power:+VSW #PWR?
 U 1 1 5E1DB6E4
 P 3200 3000
-F 0 "#PWR0130" H 3200 2850 50  0001 C CNN
+F 0 "#PWR?" H 3200 2850 50  0001 C CNN
 F 1 "+VSW" H 3215 3173 50  0000 C CNN
 F 2 "" H 3200 3000 50  0001 C CNN
@@
 $EndComp
 $Comp
-L power:-VSW #PWR0131
+L power:-VSW #PWR?
 U 1 1 5E1DBBC4
 P 3200 3600
-F 0 "#PWR0131" H 3200 3700 50  0001 C CNN
+F 0 "#PWR?" H 3200 3700 50  0001 C CNN
 F 1 "-VSW" H 3215 3773 50  0000 C CNN
 F 2 "" H 3200 3600 50  0001 C CNN
@@
 F 0 "RV26" H 4930 3346 50  0000 R CNN
 F 1 "10kLOG" H 4930 3255 50  0000 R CNN
-F 2 "4ms_Potentiometer:Pot_16mm_NoDet_RV16AF-4A" H 5000 3300 50  0001 C CNN
+F 2 "Connector_PinHeader_2.54mm:PinHeader_1x03_P2.54mm_Vertical" H 5000 3300 50  0001 C CNN
 F 3 "~" H 5000 3300 50  0001 C CNN
-F 4 "Volume" H 4800 3150 50  0000 C BNN "Label"
+F 4 "Volume" H 4750 3400 50  0000 C BNN "Label"
 	1    5000 3300
 	1    0    0    1
@@
 	5000 3150 5000 3000
 $Comp
-L power:GND #PWR0132
+L power:GND #PWR?
 U 1 1 5E1E0B28
 P 5000 3450
-F 0 "#PWR0132" H 5000 3200 50  0001 C CNN
+F 0 "#PWR?" H 5000 3200 50  0001 C CNN
 F 1 "GND" H 5005 3277 50  0000 C CNN
 F 2 "" H 5000 3450 50  0001 C CNN
@@
 $EndComp
 $Comp
-L power:+VSW #PWR0133
+L power:+VSW #PWR?
 U 1 1 5E1EC5EE
 P 7250 1400
-F 0 "#PWR0133" H 7250 1250 50  0001 C CNN
+F 0 "#PWR?" H 7250 1250 50  0001 C CNN
 F 1 "+VSW" H 7265 1573 50  0000 C CNN
 F 2 "" H 7250 1400 50  0001 C CNN
@@
 $EndComp
 $Comp
-L power:-VSW #PWR0134
+L power:-VSW #PWR?
 U 1 1 5E1EC995
 P 7250 2000
-F 0 "#PWR0134" H 7250 2100 50  0001 C CNN
-F 1 "-VSW" H 7265 2173 50  0000 C CNN
+F 0 "#PWR?" H 7250 2100 50  0001 C CNN
+F 1 "-VSW" H 7400 2150 50  0000 C CNN
 F 2 "" H 7250 2000 50  0001 C CNN
 F 3 "" H 7250 2000 50  0001 C CNN
@@
 	8050 1700 8300 1700
 $Comp
-L power:-VSW #PWR0135
+L power:-VSW #PWR?
 U 1 1 5E1F94DC
 P 7900 2850
-F 0 "#PWR0135" H 7900 2950 50  0001 C CNN
+F 0 "#PWR?" H 7900 2950 50  0001 C CNN
 F 1 "-VSW" H 7915 3023 50  0000 C CNN
 F 2 "" H 7900 2850 50  0001 C CNN
@@
 Text GLabel 2000 1550 0    50   BiDi ~ 0
 ENVELOPE
-Text GLabel 2000 1850 0    50   BiDi ~ 0
-HOLD_ON
 Wire Wire Line
 	5700 3300 5700 1800
@@
 Wire Wire Line
 	2150 4650 2050 4650
-Text GLabel 2150 4850 2    50   BiDi ~ 0
+Text GLabel 2000 1850 0    50   BiDi ~ 0
 TO_VCA_R136
-Text GLabel 2050 4850 0    50   BiDi ~ 0
-HOLD_ON
-Wire Wire Line
-	2050 4850 2150 4850
-$Comp
-L Connector:AudioJack3 J1
+$Comp
+L Connector:Conn_01x03_Male J1
 U 1 1 5ED55CB0
 P 9500 2100
-F 0 "J1" H 9220 2125 50  0000 R CNN
-F 1 "AudioJack3" H 9220 2034 50  0000 R CNN
-F 2 "4ms_Jack:EighthInch_Stereo_PJ366ST_ALT" H 9500 2100 50  0001 C CNN
+F 0 "J1" H 9400 2100 50  0000 R CNN
+F 1 "AudioJack3" H 9450 2000 50  0000 R CNN
+F 2 "Connector_PinHeader_2.54mm:PinHeader_1x03_P2.54mm_Vertical" H 9500 2100 50  0001 C CNN
 F 3 "~" H 9500 2100 50  0001 C CNN
+F 4 "STEREO OUT" H 9200 1900 50  0000 C CNN "Label"
 	1    9500 2100
 	-1   0    0    -1
@@
 	9100 1700 9300 1700
 $Comp
-L power:GND #PWR0224
+L power:GND #PWR?
 U 1 1 5ED5A487
 P 9200 2200
-F 0 "#PWR0224" H 9200 1950 50  0001 C CNN
+F 0 "#PWR?" H 9200 1950 50  0001 C CNN
 F 1 "GND" H 9205 2027 50  0000 C CNN
 F 2 "" H 9200 2200 50  0001 C CNN
@@
 	2150 5050 2050 5050
 $Comp
-L power:GND #PWR0225
+L power:GND #PWR?
 U 1 1 5EDD09AA
 P 7350 2000
-F 0 "#PWR0225" H 7350 1750 50  0001 C CNN
-F 1 "GND" H 7355 1827 50  0000 C CNN
+F 0 "#PWR?" H 7350 1750 50  0001 C CNN
+F 1 "GND" H 7450 1850 50  0000 C CNN
 F 2 "" H 7350 2000 50  0001 C CNN
 F 3 "" H 7350 2000 50  0001 C CNN
@@
 $EndComp
 $Comp
-L Connector:AudioJack2 J?
+L Connector:Conn_01x02_Male J?
 U 1 1 5EA25E4A
-P 5900 3400
+P 5900 3300
 AR Path="/5E05EC3F/5EA25E4A" Ref="J?"  Part="1"
 AR Path="/5E1B03E8/5EA25E4A" Ref="J8"  Part="1"
-F 0 "J8" H 5720 3520 50  0000 R CNN
-F 1 "AudioJack2" H 5720 3429 50  0000 R CNN
-F 2 "4ms_Jack:EighthInch_Stereo_PJ366ST_ALT" H 5900 3400 50  0001 C CNN
-F 3 "~" H 5900 3400 50  0001 C CNN
-F 4 "TRIGGER OUT" H 5720 3338 50  0000 R CNN "Label"
-	1    5900 3400
+F 0 "J8" H 5850 3350 50  0000 R CNN
+F 1 "AudioJack2" H 5850 3250 50  0000 R CNN
+F 2 "Connector_PinHeader_2.54mm:PinHeader_1x02_P2.54mm_Vertical" H 5900 3300 50  0001 C CNN
+F 3 "~" H 5900 3300 50  0001 C CNN
+F 4 "LINE OUT" H 5850 3150 50  0000 R CNN "Label"
+	1    5900 3300
 	-1   0    0    -1
 $EndComp
 $Comp
-L power:GND #PWR01
+L power:GND #PWR?
 U 1 1 5EA2727A
 P 5700 3400
-F 0 "#PWR01" H 5700 3150 50  0001 C CNN
+F 0 "#PWR?" H 5700 3150 50  0001 C CNN
 F 1 "GND" H 5705 3227 50  0000 C CNN
 F 2 "" H 5700 3400 50  0001 C CNN
@@
 	1    0    0    -1
 $EndComp
+Connection ~ 5700 3300
 $EndSCHEMATC

Commit message: Proper capacitor footprints
Parts:
- C26, C27, C28, C33: footprint Capacitor_THT:C_Disc_D5.0mm_W2.5mm_P5.00mm -> Capacitor_THT:C_Rect_L7.2mm_W2.5mm_P5.00mm_FKS2_FKP2_MKS2_MKP2
- C29, C31: value 4.7u -> 4.7u 10V
- C30: value 4.7u -> 4.7u 35V
- C32: value 4.7u -> 4.7u 25V
- C34: value 470u -> 470u 25V; footprint Capacitor_THT:CP_Radial_D5.0mm_P2.50mm -> Capacitor_THT:CP_Radial_D10.0mm_P5.00mm
Changed lines of the file:
@@
 P 2300 950
 F 0 "C30" V 2555 950 50  0000 C CNN
-F 1 "4.7u" V 2464 950 50  0000 C CNN
+F 1 "4.7u 35V" V 2464 950 50  0000 C CNN
 F 2 "Capacitor_THT:CP_Radial_D5.0mm_P2.50mm" H 2338 800 50  0001 C CNN
 F 3 "~" H 2300 950 50  0001 C CNN
@@
 F 0 "C26" V 1048 2650 50  0000 C CNN
 F 1 "220n" V 1139 2650 50  0000 C CNN
-F 2 "Capacitor_THT:C_Disc_D5.0mm_W2.5mm_P5.00mm" H 1338 2500 50  0001 C CNN
+F 2 "Capacitor_THT:C_Rect_L7.2mm_W2.5mm_P5.00mm_FKS2_FKP2_MKS2_MKP2" H 1338 2500 50  0001 C CNN
 F 3 "~" H 1300 2650 50  0001 C CNN
 	1    1300 2650
@@
 F 0 "C27" V 1552 3050 50  0000 C CNN
 F 1 "220n" V 1461 3050 50  0000 C CNN
-F 2 "Capacitor_THT:C_Disc_D5.0mm_W2.5mm_P5.00mm" H 1338 2900 50  0001 C CNN
+F 2 "Capacitor_THT:C_Rect_L7.2mm_W2.5mm_P5.00mm_FKS2_FKP2_MKS2_MKP2" H 1338 2900 50  0001 C CNN
 F 3 "~" H 1300 3050 50  0001 C CNN
 	1    1300 3050
@@
 F 0 "C28" V 1552 3450 50  0000 C CNN
 F 1 "220n" V 1461 3450 50  0000 C CNN
-F 2 "Capacitor_THT:C_Disc_D5.0mm_W2.5mm_P5.00mm" H 1338 3300 50  0001 C CNN
+F 2 "Capacitor_THT:C_Rect_L7.2mm_W2.5mm_P5.00mm_FKS2_FKP2_MKS2_MKP2" H 1338 3300 50  0001 C CNN
 F 3 "~" H 1300 3450 50  0001 C CNN
 	1    1300 3450
@@
 P 4600 2500
 F 0 "C29" V 4855 2500 50  0000 C CNN
-F 1 "4.7u" V 4764 2500 50  0000 C CNN
+F 1 "4.7u 10V" V 4764 2500 50  0000 C CNN
 F 2 "Capacitor_THT:CP_Radial_D5.0mm_P2.50mm" H 4638 2350 50  0001 C CNN
 F 3 "~" H 4600 2500 50  0001 C CNN
@@
 P 6500 1800
 F 0 "C31" V 6245 1800 50  0000 C CNN
-F 1 "4.7u" V 6336 1800 50  0000 C CNN
+F 1 "4.7u 10V" V 6336 1800 50  0000 C CNN
 F 2 "Capacitor_THT:CP_Radial_D5.0mm_P2.50mm" H 6538 1650 50  0001 C CNN
 F 3 "~" H 6500 1800 50  0001 C CNN
@@
 P 8450 1700
 F 0 "C34" V 8705 1700 50  0000 C CNN
-F 1 "470u" V 8614 1700 50  0000 C CNN
-F 2 "Capacitor_THT:CP_Radial_D5.0mm_P2.50mm" H 8488 1550 50  0001 C CNN
+F 1 "470u 25V" V 8614 1700 50  0000 C CNN
+F 2 "Capacitor_THT:CP_Radial_D10.0mm_P5.00mm" H 8488 1550 50  0001 C CNN
 F 3 "~" H 8450 1700 50  0001 C CNN
 	1    8450 1700
@@
 P 7750 2300
 F 0 "C32" H 7868 2346 50  0000 L CNN
-F 1 "4.7u" H 7868 2255 50  0000 L CNN
+F 1 "4.7u 25V" H 7868 2255 50  0000 L CNN
 F 2 "Capacitor_THT:CP_Radial_D5.0mm_P2.50mm" H 7788 2150 50  0001 C CNN
 F 3 "~" H 7750 2300 50  0001 C CNN
@@
 F 0 "C33" H 8165 2596 50  0000 L CNN
 F 1 "100n" H 8165 2505 50  0000 L CNN
-F 2 "Capacitor_THT:C_Disc_D5.0mm_W2.5mm_P5.00mm" H 8088 2400 50  0001 C CNN
+F 2 "Capacitor_THT:C_Rect_L7.2mm_W2.5mm_P5.00mm_FKS2_FKP2_MKS2_MKP2" H 8088 2400 50  0001 C CNN
 F 3 "~" H 8050 2550 50  0001 C CNN
 	1    8050 2550
