File: microsynth/VCO2.sch (KiCad schematic (older format))
At the start: 31 parts, among them IC5 TL074, U14 4016, U15 LF355, U16 LM741, U17 LM741, U18 LM741

Commit message: Footprints
Parts:
- U5: renamed from IC5; footprint (none) -> Package_DIP:DIP-14_W7.62mm
Other:
- moved on the sheet: C18, C19, C20, R142, R143, R82, R85, R86, R87, R88, R89, R90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

Commit message: Footprints 2
Parts:
- C18, C19, C20: footprint (none) -> Capacitor_THT:C_Disc_D5.0mm_W2.5mm_P5.00mm
- R94_1: footprint (none) -> Resistor_THT:R_Axial_DIN0207_L6.3mm_D2.5mm_P10.16mm_Horizontal
- U14: footprint (none) -> Package_DIP:DIP-14_W7.62mm_LongPads
- U15, U16, U17, U18: footprint (none) -> Package_DIP:DIP-8_W7.62mm_LongPads
Changed lines of the file:
@@
 F 0 "U17" H 4344 5454 50  0000 L CNN
 F 1 "LM741" H 4344 5545 50  0000 L CNN
-F 2 "" H 4050 5550 50  0001 C CNN
+F 2 "Package_DIP:DIP-8_W7.62mm_LongPads" H 4050 5550 50  0001 C CNN
 F 3 "http://www.ti.com/lit/ds/symlink/lm741.pdf" H 4150 5650 50  0001 C CNN
 	1    4000 5500
@@
 F 0 "U16" H 3044 5454 50  0000 L CNN
 F 1 "LM741" H 3044 5545 50  0000 L CNN
-F 2 "" H 2750 5550 50  0001 C CNN
+F 2 "Package_DIP:DIP-8_W7.62mm_LongPads" H 2750 5550 50  0001 C CNN
 F 3 "http://www.ti.com/lit/ds/symlink/lm741.pdf" H 2850 5650 50  0001 C CNN
 	1    2700 5500
@@
 F 0 "U18" H 4144 2954 50  0000 L CNN
 F 1 "LM741" H 4144 3045 50  0000 L CNN
-F 2 "" H 3850 3050 50  0001 C CNN
+F 2 "Package_DIP:DIP-8_W7.62mm_LongPads" H 3850 3050 50  0001 C CNN
 F 3 "http://www.ti.com/lit/ds/symlink/lm741.pdf" H 3950 3150 50  0001 C CNN
 	1    3800 3000
@@
 F 0 "C20" V 2448 5100 50  0000 C CNN
 F 1 "10n" V 2539 5100 50  0000 C CNN
-F 2 "" H 2738 4950 50  0001 C CNN
+F 2 "Capacitor_THT:C_Disc_D5.0mm_W2.5mm_P5.00mm" H 2738 4950 50  0001 C CNN
 F 3 "~" H 2700 5100 50  0001 C CNN
 	1    2700 5100
@@
 F 0 "R94_1" H 4070 4396 50  0000 L CNN
 F 1 "1M" H 4070 4305 50  0000 L CNN
-F 2 "" V 3930 4350 50  0001 C CNN
+F 2 "Resistor_THT:R_Axial_DIN0207_L6.3mm_D2.5mm_P10.16mm_Horizontal" V 3930 4350 50  0001 C CNN
 F 3 "~" H 4000 4350 50  0001 C CNN
 	1    4000 4350
@@
 F 0 "C19" V 1148 4350 50  0000 C CNN
 F 1 "15n" V 1239 4350 50  0000 C CNN
-F 2 "" H 1438 4200 50  0001 C CNN
+F 2 "Capacitor_THT:C_Disc_D5.0mm_W2.5mm_P5.00mm" H 1438 4200 50  0001 C CNN
 F 3 "~" H 1400 4350 50  0001 C CNN
 	1    1400 4350
@@
 F 0 "C18" V 2148 2600 50  0000 C CNN
 F 1 "10n" V 2239 2600 50  0000 C CNN
-F 2 "" H 2438 2450 50  0001 C CNN
+F 2 "Capacitor_THT:C_Disc_D5.0mm_W2.5mm_P5.00mm" H 2438 2450 50  0001 C CNN
 F 3 "~" H 2400 2600 50  0001 C CNN
 	1    2400 2600
@@
 F 0 "U15" H 2494 2954 50  0000 L CNN
 F 1 "LF355" H 2494 3045 50  0000 L CNN
-F 2 "" H 2200 3050 50  0001 C CNN
+F 2 "Package_DIP:DIP-8_W7.62mm_LongPads" H 2200 3050 50  0001 C CNN
 F 3 "http://www.ti.com/lit/ds/symlink/lf357.pdf" H 2300 3150 50  0001 C CNN
 	1    2150 3000
@@
 F 0 "U14" V 1304 3672 50  0000 R CNN
 F 1 "4016" V 1395 3672 50  0000 R CNN
-F 2 "" H 1350 3800 50  0001 C CNN
+F 2 "Package_DIP:DIP-14_W7.62mm_LongPads" H 1350 3800 50  0001 C CNN
 F 3 "http://www.ti.com/lit/ds/symlink/cd4016b.pdf" H 1350 3800 50  0001 C CNN
 	1    1350 3800
@@
 F 0 "U14" H 2950 4577 50  0000 C CNN
 F 1 "4016" H 2950 4486 50  0000 C CNN
-F 2 "" H 2950 4750 50  0001 C CNN
+F 2 "Package_DIP:DIP-14_W7.62mm_LongPads" H 2950 4750 50  0001 C CNN
 F 3 "http://www.ti.com/lit/ds/symlink/cd4016b.pdf" H 2950 4750 50  0001 C CNN
 	4    2950 4750

Commit message: Hacking together the footprints
Parts:
- RV16: value 1k -> 1kLIN; footprint (none) -> 4ms_Potentiometer:Pot_16mm_NoDet_RV16AF-4A
- RV17, RV19: footprint (none) -> Potentiometers:Potentiometer_Trimmer_Bourns_PV36W
- RV18: value 100k -> 100kLIN; footprint (none) -> 4ms_Potentiometer:Pot_16mm_NoDet_RV16AF-4A
Changed lines of the file:
@@
 P 1100 1750
 F 0 "RV16" H 1030 1659 50  0000 R CNN
-F 1 "1k" H 1030 1750 50  0000 R CNN
-F 2 "" H 1100 1750 50  0001 C CNN
+F 1 "1kLIN" H 1030 1750 50  0000 R CNN
+F 2 "4ms_Potentiometer:Pot_16mm_NoDet_RV16AF-4A" H 1100 1750 50  0001 C CNN
 F 3 "~" H 1100 1750 50  0001 C CNN
 F 4 "VCO2 FREQ" H 1030 1841 50  0000 R CNN "Label"
@@
 P 4000 3900
 F 0 "RV18" H 3930 3854 50  0000 R CNN
-F 1 "100k" H 3930 3945 50  0000 R CNN
-F 2 "" H 4000 3900 50  0001 C CNN
+F 1 "100kLIN" H 3930 3945 50  0000 R CNN
+F 2 "4ms_Potentiometer:Pot_16mm_NoDet_RV16AF-4A" H 4000 3900 50  0001 C CNN
 F 3 "~" H 4000 3900 50  0001 C CNN
 	1    4000 3900
@@
 F 0 "RV19" H 880 4696 50  0000 R CNN
 F 1 "100k" H 880 4605 50  0000 R CNN
-F 2 "" H 950 4650 50  0001 C CNN
+F 2 "Potentiometers:Potentiometer_Trimmer_Bourns_PV36W" H 950 4650 50  0001 C CNN
 F 3 "~" H 950 4650 50  0001 C CNN
 	1    950  4650
@@
 F 0 "RV17" V 1993 2200 50  0000 C CNN
 F 1 "10k" V 2084 2200 50  0000 C CNN
-F 2 "" H 2200 2200 50  0001 C CNN
+F 2 "Potentiometers:Potentiometer_Trimmer_Bourns_PV36W" H 2200 2200 50  0001 C CNN
 F 3 "~" H 2200 2200 50  0001 C CNN
 	1    2200 2200

Commit message: All components placed on PCB
Parts:
- renumbered R94 to R84, R94_1 to R94
Changed lines of the file:
@@
 U 1 1 5E2D86CD
 P 4000 5500
-F 0 "U17" H 4344 5454 50  0000 L CNN
-F 1 "LM741" H 4344 5545 50  0000 L CNN
+F 0 "U17" H 3900 5550 50  0000 L CNN
+F 1 "LM741" H 4000 5650 50  0000 L CNN
 F 2 "Package_DIP:DIP-8_W7.62mm_LongPads" H 4050 5550 50  0001 C CNN
 F 3 "http://www.ti.com/lit/ds/symlink/lm741.pdf" H 4150 5650 50  0001 C CNN
@@
 U 1 1 5E2D9591
 P 2700 5500
-F 0 "U16" H 3044 5454 50  0000 L CNN
-F 1 "LM741" H 3044 5545 50  0000 L CNN
+F 0 "U16" H 2600 5500 50  0000 L CNN
+F 1 "LM741" H 2650 5650 50  0000 L CNN
 F 2 "Package_DIP:DIP-8_W7.62mm_LongPads" H 2750 5550 50  0001 C CNN
 F 3 "http://www.ti.com/lit/ds/symlink/lm741.pdf" H 2850 5650 50  0001 C CNN
@@
 U 1 1 5E2D9E6C
 P 3800 3000
-F 0 "U18" H 4144 2954 50  0000 L CNN
-F 1 "LM741" H 4144 3045 50  0000 L CNN
+F 0 "U18" H 3700 3000 50  0000 L CNN
+F 1 "LM741" H 3700 3200 50  0000 L CNN
 F 2 "Package_DIP:DIP-8_W7.62mm_LongPads" H 3850 3050 50  0001 C CNN
 F 3 "http://www.ti.com/lit/ds/symlink/lm741.pdf" H 3950 3150 50  0001 C CNN
@@
 $EndComp
 $Comp
-L Device:R R94
+L Device:R R84
 U 1 1 5E2F2B85
 P 900 3100
-F 0 "R94" H 970 3146 50  0000 L CNN
+F 0 "R84" H 970 3146 50  0000 L CNN
 F 1 "10k" H 970 3055 50  0000 L CNN
 F 2 "Resistor_THT:R_Axial_DIN0207_L6.3mm_D2.5mm_P10.16mm_Horizontal" V 830 3100 50  0001 C CNN
@@
 $EndComp
 $Comp
-L Device:R R94_1
+L Device:R R94
 U 1 1 5E2F5D7A
 P 4000 4350
-F 0 "R94_1" H 4070 4396 50  0000 L CNN
+F 0 "R94" H 4070 4396 50  0000 L CNN
 F 1 "1M" H 4070 4305 50  0000 L CNN
 F 2 "Resistor_THT:R_Axial_DIN0207_L6.3mm_D2.5mm_P10.16mm_Horizontal" V 3930 4350 50  0001 C CNN
@@
 U 1 1 5E322633
 P 2150 3000
-F 0 "U15" H 2494 2954 50  0000 L CNN
-F 1 "LF355" H 2494 3045 50  0000 L CNN
+F 0 "U15" H 2050 3000 50  0000 L CNN
+F 1 "LF355" H 2100 3150 50  0000 L CNN
 F 2 "Package_DIP:DIP-8_W7.62mm_LongPads" H 2200 3050 50  0001 C CNN
 F 3 "http://www.ti.com/lit/ds/symlink/lf357.pdf" H 2300 3150 50  0001 C CNN

Commit message: Laying out pcb
Parts:
- removed U5: TL074, Package_DIP:DIP-14_W7.62mm, symbol Amplifier_Operational:TL074
- added U5: LF347, Package_DIP:DIP-14_W7.62mm_LongPads, symbol Amplifier_Operational:LF347
Connections:
- net S5_VCO2: now also U5.8
- net VCO2_TRI: now also U5.9 (-)
- net at R88.1, R89.2: now also U5.10 (+)
- net at C18.2, R87.1, U15.2 (-): no longer RV17.1, U15.5 (NULL)
- new net: RV17.1, U15.5 (NULL)
Other:
- moved on the sheet: C18
Changed lines of the file:
@@
 $EndDescr
-$Comp
-L Amplifier_Operational:TL074 IC?
-U 3 1 5E2D3C59
-P 2900 3100
-AR Path="/5E222DC1/5E2D3C59" Ref="IC?"  Part="3"
-AR Path="/5E2BE1AD/5E2D3C59" Ref="U5"  Part="3"
-F 0 "U5" H 2900 2733 50  0000 C CNN
-F 1 "TL074" H 2900 2824 50  0000 C CNN
-F 2 "Package_DIP:DIP-14_W7.62mm" H 2850 3200 50  0001 C CNN
-F 3 "http://www.ti.com/lit/ds/symlink/tl071.pdf" H 2950 3300 50  0001 C CNN
-	3    2900 3100
-	1    0    0    1
-$EndComp
 $Comp
 L Amplifier_Operational:LM741 U17
@@
 L Device:C C18
 U 1 1 5E3101FB
-P 2400 2600
-F 0 "C18" V 2148 2600 50  0000 C CNN
-F 1 "10n" V 2239 2600 50  0000 C CNN
-F 2 "Capacitor_THT:C_Disc_D5.0mm_W2.5mm_P5.00mm" H 2438 2450 50  0001 C CNN
-F 3 "~" H 2400 2600 50  0001 C CNN
-	1    2400 2600
-	0    1    1    0
-$EndComp
-Wire Wire Line
-	2250 2600 1850 2600
-Wire Wire Line
-	1850 2600 1850 2800
+P 2400 1850
+F 0 "C18" V 2148 1850 50  0000 C CNN
+F 1 "10n" V 2239 1850 50  0000 C CNN
+F 2 "Capacitor_THT:C_Disc_D5.0mm_W2.5mm_P5.00mm" H 2438 1700 50  0001 C CNN
+F 3 "~" H 2400 1850 50  0001 C CNN
+	1    2400 1850
+	0    1    1    0
+$EndComp
 Wire Wire Line
 	1850 2800 1750 2800
@@
 Wire Wire Line
 	2400 2350 2250 2350
-Wire Wire Line
-	2250 2350 2250 2600
 $Comp
 L power:-VSW #PWR0162
@@
 Wire Wire Line
 	3250 850  3250 3100
-Connection ~ 2250 2600
-Wire Wire Line
-	2250 2600 2250 2700
 $Comp
 L power:-VSW #PWR0164
@@
 	4300 5500 4350 5500
 Connection ~ 4350 5500
+$Comp
+L Amplifier_Operational:LF347 U?
+U 3 1 5E9127FD
+P 2900 3100
+AR Path="/5E8C1704/5E9127FD" Ref="U?"  Part="3"
+AR Path="/5E2BE1AD/5E9127FD" Ref="U5"  Part="3"
+F 0 "U5" H 2900 2700 50  0000 C CNN
+F 1 "LF347" H 2900 2800 50  0000 C CNN
+F 2 "Package_DIP:DIP-14_W7.62mm_LongPads" H 2850 3200 50  0001 C CNN
+F 3 "https://www.ti.com/lit/ds/symlink/lf147.pdf" H 2950 3300 50  0001 C CNN
+	3    2900 3100
+	1    0    0    1
+$EndComp
+Wire Wire Line
+	2250 2350 2250 2700
+Wire Wire Line
+	2550 2600 2550 1850
+Wire Wire Line
+	1850 1850 2250 1850
+Wire Wire Line
+	1850 1850 1850 2800
 $EndSCHEMATC

Commit message: Laying out pcb ...
Connections:
- net GND: now also RV19.1; no longer RV19.3
- net at C19.2: now also RV19.3; no longer RV19.1
Changed lines of the file:
@@
 F 3 "~" H 950 4650 50  0001 C CNN
 	1    950  4650
-	1    0    0    -1
+	1    0    0    1
 $EndComp
 $Comp

Commit message: Proper capacitor footprints
Parts:
- C18, C20: footprint Capacitor_THT:C_Disc_D5.0mm_W2.5mm_P5.00mm -> Capacitor_THT:C_Rect_L7.2mm_W2.5mm_P5.00mm_FKS2_FKP2_MKS2_MKP2
- C19: footprint Capacitor_THT:C_Disc_D5.0mm_W2.5mm_P5.00mm -> Capacitor_THT:C_Rect_L7.2mm_W3.5mm_P5.00mm_FKS2_FKP2_MKS2_MKP2
Changed lines of the file:
@@
 F 0 "C20" V 2448 5100 50  0000 C CNN
 F 1 "10n" V 2539 5100 50  0000 C CNN
-F 2 "Capacitor_THT:C_Disc_D5.0mm_W2.5mm_P5.00mm" H 2738 4950 50  0001 C CNN
+F 2 "Capacitor_THT:C_Rect_L7.2mm_W2.5mm_P5.00mm_FKS2_FKP2_MKS2_MKP2" H 2738 4950 50  0001 C CNN
 F 3 "~" H 2700 5100 50  0001 C CNN
 	1    2700 5100
@@
 F 0 "C19" V 1148 4350 50  0000 C CNN
 F 1 "15n" V 1239 4350 50  0000 C CNN
-F 2 "Capacitor_THT:C_Disc_D5.0mm_W2.5mm_P5.00mm" H 1438 4200 50  0001 C CNN
+F 2 "Capacitor_THT:C_Rect_L7.2mm_W3.5mm_P5.00mm_FKS2_FKP2_MKS2_MKP2" H 1438 4200 50  0001 C CNN
 F 3 "~" H 1400 4350 50  0001 C CNN
 	1    1400 4350
@@
 F 0 "C18" V 2148 1850 50  0000 C CNN
 F 1 "10n" V 2239 1850 50  0000 C CNN
-F 2 "Capacitor_THT:C_Disc_D5.0mm_W2.5mm_P5.00mm" H 2438 1700 50  0001 C CNN
+F 2 "Capacitor_THT:C_Rect_L7.2mm_W2.5mm_P5.00mm_FKS2_FKP2_MKS2_MKP2" H 2438 1700 50  0001 C CNN
 F 3 "~" H 2400 1850 50  0001 C CNN
 	1    2400 1850
