File: microsynth/VCO2.sch (KiCad schematic (older format))
At the start: 31 parts, among them U14 4016, U15 LF355, U16 LM741, U17 LM741, U18 LM741, U5 LF347

Commit message: Label pots
Parts:
- RV18: Label (none) -> VCO2 PWM
Changed lines of the file:
@@
 F 2 "4ms_Potentiometer:Pot_16mm_NoDet_RV16AF-4A" H 4000 3900 50  0001 C CNN
 F 3 "~" H 4000 3900 50  0001 C CNN
+F 4 "VCO2 PWM" H 3750 4050 50  0000 C CNN "Label"
 	1    4000 3900
 	-1   0    0    1

Commit message: Clean up repo
Parts:
- U5: symbol Amplifier_Operational:LF347 -> microsynth-rescue:LF347-Amplifier_Operational
Changed lines of the file:
@@
 Connection ~ 4350 5500
 $Comp
-L Amplifier_Operational:LF347 U?
+L microsynth-rescue:LF347-Amplifier_Operational U?
 U 3 1 5E9127FD
 P 2900 3100
 AR Path="/5E8C1704/5E9127FD" Ref="U?"  Part="3"
 AR Path="/5E2BE1AD/5E9127FD" Ref="U5"  Part="3"
+AR Path="/5E9127FD" Ref="U5"  Part="3"
 F 0 "U5" H 2900 2700 50  0000 C CNN
 F 1 "LF347" H 2900 2800 50  0000 C CNN

Commit message: Replace dodgy parts 1458, 4136 & LF351s
Parts:
- removed U15: LF355, Package_DIP:DIP-8_W7.62mm_LongPads, symbol Amplifier_Operational:LF355
- removed U5: LF347, Package_DIP:DIP-14_W7.62mm_LongPads, symbol microsynth-rescue:LF347-Amplifier_Operational
- added U15: LF351, Package_DIP:DIP-8_W7.62mm_LongPads, symbol pe_microsynth:LF351
- added U5: LF347, Package_DIP:DIP-14_W7.62mm_LongPads, symbol pe_microsynth:LF347
Connections:
- net +VSW: now also U15.7 (V+)
- net -VSW: now also U15.4 (V-)
- net S5_VCO2: now also U5.8
- net VCO2_TRI: now also U15.6, U5.9 (-)
- net at C18.2, R87.1: now also U15.2 (-)
- net at R84.2, R85.1: now also U15.3 (+)
- net at R88.1, R89.2: now also U5.10 (+)
- net at RV17.3: now also U15.1 (NULL)
- net at RV17.1: now also U15.5 (NULL)
Changed lines of the file:
@@
 Wire Wire Line
 	3600 5600 3700 5600
-$Comp
-L Amplifier_Operational:LF355 U15
-U 1 1 5E322633
-P 2150 3000
-F 0 "U15" H 2050 3000 50  0000 L CNN
-F 1 "LF355" H 2100 3150 50  0000 L CNN
-F 2 "Package_DIP:DIP-8_W7.62mm_LongPads" H 2200 3050 50  0001 C CNN
-F 3 "http://www.ti.com/lit/ds/symlink/lf357.pdf" H 2300 3150 50  0001 C CNN
-	1    2150 3000
-	1    0    0    1
-$EndComp
 Wire Wire Line
 	1850 2900 1850 2800
@@
 	4300 5500 4350 5500
 Connection ~ 4350 5500
-$Comp
-L microsynth-rescue:LF347-Amplifier_Operational U?
-U 3 1 5E9127FD
+Wire Wire Line
+	2250 2350 2250 2700
+Wire Wire Line
+	2550 2600 2550 1850
+Wire Wire Line
+	1850 1850 2250 1850
+Wire Wire Line
+	1850 1850 1850 2800
+$Comp
+L pe_microsynth:LF347 U?
+U 3 1 5EBF1DEA
 P 2900 3100
-AR Path="/5E8C1704/5E9127FD" Ref="U?"  Part="3"
-AR Path="/5E2BE1AD/5E9127FD" Ref="U5"  Part="3"
-AR Path="/5E9127FD" Ref="U5"  Part="3"
-F 0 "U5" H 2900 2700 50  0000 C CNN
-F 1 "LF347" H 2900 2800 50  0000 C CNN
+AR Path="/5E8C1704/5EBF1DEA" Ref="U?"  Part="3"
+AR Path="/5E2BE1AD/5EBF1DEA" Ref="U5"  Part="3"
+F 0 "U5" H 2850 3100 50  0000 C CNN
+F 1 "LF347" H 2900 2900 50  0000 C CNN
 F 2 "Package_DIP:DIP-14_W7.62mm_LongPads" H 2850 3200 50  0001 C CNN
-F 3 "https://www.ti.com/lit/ds/symlink/lf147.pdf" H 2950 3300 50  0001 C CNN
+F 3 "https://www.bitsbox.co.uk/data/analog/LF347.pdf" H 2950 3300 50  0001 C CNN
 	3    2900 3100
 	1    0    0    1
 $EndComp
-Wire Wire Line
-	2250 2350 2250 2700
-Wire Wire Line
-	2550 2600 2550 1850
-Wire Wire Line
-	1850 1850 2250 1850
-Wire Wire Line
-	1850 1850 1850 2800
+$Comp
+L pe_microsynth:LF351 U15
+U 1 1 5EC56017
+P 2150 3000
+F 0 "U15" H 2050 3000 50  0000 L CNN
+F 1 "LF351" H 2150 3150 50  0000 L CNN
+F 2 "Package_DIP:DIP-8_W7.62mm_LongPads" H 2200 3050 50  0001 C CNN
+F 3 "https://www.bitsbox.co.uk/data/opamps/lf351.pdf" H 2300 3150 50  0001 C CNN
+	1    2150 3000
+	1    0    0    1
+$EndComp
 $EndSCHEMATC

Commit message: Consolidate all(?) switches
Parts:
- RV16, RV18: footprint 4ms_Potentiometer:Pot_16mm_NoDet_RV16AF-4A -> microsynth:Pot_16mm_NoDet_RV16AF-4A
Changed lines of the file:
@@
 F 0 "RV16" H 1030 1659 50  0000 R CNN
 F 1 "1kLIN" H 1030 1750 50  0000 R CNN
-F 2 "4ms_Potentiometer:Pot_16mm_NoDet_RV16AF-4A" H 1100 1750 50  0001 C CNN
+F 2 "microsynth:Pot_16mm_NoDet_RV16AF-4A" H 1100 1750 50  0001 C CNN
 F 3 "~" H 1100 1750 50  0001 C CNN
 F 4 "VCO2 FREQ" H 1030 1841 50  0000 R CNN "Label"
@@
 F 0 "RV18" H 3930 3854 50  0000 R CNN
 F 1 "100kLIN" H 3930 3945 50  0000 R CNN
-F 2 "4ms_Potentiometer:Pot_16mm_NoDet_RV16AF-4A" H 4000 3900 50  0001 C CNN
+F 2 "microsynth:Pot_16mm_NoDet_RV16AF-4A" H 4000 3900 50  0001 C CNN
 F 3 "~" H 4000 3900 50  0001 C CNN
 F 4 "VCO2 PWM" H 3750 4050 50  0000 C CNN "Label"

Commit message: Replace IC1 with LM348, update component values
Parts:
- R91: value 1k -> 6k8
- R92: value 220 -> 1k5
Changed lines of the file:
@@
 P 4300 3000
 F 0 "R91" V 4093 3000 50  0000 C CNN
-F 1 "1k" V 4184 3000 50  0000 C CNN
+F 1 "6k8" V 4184 3000 50  0000 C CNN
 F 2 "Resistor_THT:R_Axial_DIN0207_L6.3mm_D2.5mm_P10.16mm_Horizontal" V 4230 3000 50  0001 C CNN
 F 3 "~" H 4300 3000 50  0001 C CNN
@@
 P 4500 3300
 F 0 "R92" H 4570 3346 50  0000 L CNN
-F 1 "220" H 4570 3255 50  0000 L CNN
+F 1 "1k5" H 4570 3255 50  0000 L CNN
 F 2 "Resistor_THT:R_Axial_DIN0207_L6.3mm_D2.5mm_P10.16mm_Horizontal" V 4430 3300 50  0001 C CNN
 F 3 "~" H 4500 3300 50  0001 C CNN
