File: microsynth/power.sch (KiCad schematic (older format))
At the start: 10 parts, among them J2 Conn_01x03_Male, J3 Conn_01x06_Male, J4 Conn_01x04_Male

Commit message: Replace power connector with 4 pin molex p3.96
Parts:
- removed J2: Conn_01x03_Male, Connector_PinHeader_2.54mm:PinHeader_1x03_P2.54mm_Vertical, symbol Connector:Conn_01x03_Male
- added J2: Conn_01x04_Male, Connector_Molex:Molex_KK-396_A-41791-0004_1x04_P3.96mm_Vertical, symbol Connector:Conn_01x04_Male
Connections:
- wire segments 8 -> 11
Changed lines of the file:
@@
 L power:PWR_FLAG #FLG?
 U 1 1 5E0610BE
-P 7150 1500
-F 0 "#FLG?" H 7150 1575 50  0001 C CNN
-F 1 "PWR_FLAG" H 7150 1673 50  0000 C CNN
-F 2 "" H 7150 1500 50  0001 C CNN
-F 3 "~" H 7150 1500 50  0001 C CNN
-	1    7150 1500
+P 7150 1600
+F 0 "#FLG?" H 7150 1675 50  0001 C CNN
+F 1 "PWR_FLAG" H 7150 1773 50  0000 C CNN
+F 2 "" H 7150 1600 50  0001 C CNN
+F 3 "~" H 7150 1600 50  0001 C CNN
+	1    7150 1600
 	-1   0    0    1
 $EndComp
@@
 TRIG_OUT_TO_SEQ_SKT
 $Comp
-L Connector:Conn_01x03_Male J2
-U 1 1 5F1FC317
-P 6500 1400
-F 0 "J2" H 6650 1700 50  0000 C CNN
-F 1 "Conn_01x03_Male" H 6650 1600 50  0000 C CNN
-F 2 "Connector_PinHeader_2.54mm:PinHeader_1x03_P2.54mm_Vertical" H 6500 1400 50  0001 C CNN
-F 3 "~" H 6500 1400 50  0001 C CNN
-	1    6500 1400
-	1    0    0    -1
-$EndComp
-$Comp
 L Connector:Conn_01x04_Male J4
 U 1 1 5F1FE242
@@
 L power:-VSW #PWR?
 U 1 1 5F231D96
-P 6850 1500
-F 0 "#PWR?" H 6850 1600 50  0001 C CNN
-F 1 "-VSW" H 6865 1673 50  0000 C CNN
-F 2 "" H 6850 1500 50  0001 C CNN
-F 3 "" H 6850 1500 50  0001 C CNN
-	1    6850 1500
+P 6850 1600
+F 0 "#PWR?" H 6850 1700 50  0001 C CNN
+F 1 "-VSW" H 6865 1773 50  0000 C CNN
+F 2 "" H 6850 1600 50  0001 C CNN
+F 3 "" H 6850 1600 50  0001 C CNN
+	1    6850 1600
 	-1   0    0    1
 $EndComp
 Wire Wire Line
-	6700 1500 6850 1500
+	6700 1600 6850 1600
 $Comp
 L power:GND #PWR?
@@
 $EndComp
 Wire Wire Line
-	7450 1400 6700 1400
+	7450 1400 7050 1400
 $Comp
 L power:+VSW #PWR?
@@
 $EndComp
 Wire Wire Line
-	7150 1500 6850 1500
-Connection ~ 6850 1500
+	7150 1600 6850 1600
+Connection ~ 6850 1600
 Wire Wire Line
 	7450 1300 7050 1300
@@
 Wire Wire Line
 	6850 3100 5900 3100
+$Comp
+L Connector:Conn_01x04_Male J2
+U 1 1 5F5AB22D
+P 6500 1400
+F 0 "J2" H 6650 1700 50  0000 C CNN
+F 1 "Conn_01x04_Male" H 6650 1600 50  0000 C CNN
+F 2 "Connector_Molex:Molex_KK-396_A-41791-0004_1x04_P3.96mm_Vertical" H 6500 1400 50  0001 C CNN
+F 3 "~" H 6500 1400 50  0001 C CNN
+	1    6500 1400
+	1    0    0    -1
+$EndComp
+Wire Wire Line
+	7050 1500 7050 1400
+Wire Wire Line
+	6700 1500 7050 1500
+Connection ~ 7050 1400
+Wire Wire Line
+	7050 1400 6700 1400
 $EndSCHEMATC

Commit message: Replace power connector (again) with a plug-in style, remove redundant global label
Parts:
- J2: footprint Connector_Molex:Molex_KK-396_A-41791-0004_1x04_P3.96mm_Vertical -> Connector_Phoenix_MSTB:PhoenixContact_MSTBA_2,5_3-G_1x03_P5.00mm_Horizontal; symbol Connector:Conn_01x04_Male -> Connector:Conn_01x03_Male
Connections:
- wire segments 11 -> 8
Changed lines of the file:
@@
 L power:PWR_FLAG #FLG?
 U 1 1 5E0610BE
-P 7150 1600
-F 0 "#FLG?" H 7150 1675 50  0001 C CNN
-F 1 "PWR_FLAG" H 7150 1773 50  0000 C CNN
-F 2 "" H 7150 1600 50  0001 C CNN
-F 3 "~" H 7150 1600 50  0001 C CNN
-	1    7150 1600
+P 7150 1500
+F 0 "#FLG?" H 7150 1575 50  0001 C CNN
+F 1 "PWR_FLAG" H 7150 1673 50  0000 C CNN
+F 2 "" H 7150 1500 50  0001 C CNN
+F 3 "~" H 7150 1500 50  0001 C CNN
+	1    7150 1500
 	-1   0    0    1
 $EndComp
@@
 L power:-VSW #PWR?
 U 1 1 5F231D96
-P 6850 1600
-F 0 "#PWR?" H 6850 1700 50  0001 C CNN
-F 1 "-VSW" H 6865 1773 50  0000 C CNN
-F 2 "" H 6850 1600 50  0001 C CNN
-F 3 "" H 6850 1600 50  0001 C CNN
-	1    6850 1600
+P 6850 1500
+F 0 "#PWR?" H 6850 1600 50  0001 C CNN
+F 1 "-VSW" H 6865 1673 50  0000 C CNN
+F 2 "" H 6850 1500 50  0001 C CNN
+F 3 "" H 6850 1500 50  0001 C CNN
+	1    6850 1500
 	-1   0    0    1
 $EndComp
 Wire Wire Line
-	6700 1600 6850 1600
+	6700 1500 6850 1500
 $Comp
 L power:GND #PWR?
@@
 	1    0    0    -1
 $EndComp
-Wire Wire Line
-	7450 1400 7050 1400
 $Comp
 L power:+VSW #PWR?
@@
 $EndComp
 Wire Wire Line
-	7150 1600 6850 1600
-Connection ~ 6850 1600
+	7150 1500 6850 1500
+Connection ~ 6850 1500
 Wire Wire Line
 	7450 1300 7050 1300
@@
 	6850 3100 5900 3100
 $Comp
-L Connector:Conn_01x04_Male J2
+L Connector:Conn_01x03_Male J2
 U 1 1 5F5AB22D
 P 6500 1400
-F 0 "J2" H 6650 1700 50  0000 C CNN
-F 1 "Conn_01x04_Male" H 6650 1600 50  0000 C CNN
-F 2 "Connector_Molex:Molex_KK-396_A-41791-0004_1x04_P3.96mm_Vertical" H 6500 1400 50  0001 C CNN
+F 0 "J2" H 6450 1300 50  0000 R CNN
+F 1 "Conn_01x04_Male" H 6450 1400 50  0000 R CNN
+F 2 "Connector_Phoenix_MSTB:PhoenixContact_MSTBA_2,5_3-G_1x03_P5.00mm_Horizontal" H 6500 1400 50  0001 C CNN
 F 3 "~" H 6500 1400 50  0001 C CNN
 	1    6500 1400
-	1    0    0    -1
-$EndComp
-Wire Wire Line
-	7050 1500 7050 1400
-Wire Wire Line
-	6700 1500 7050 1500
-Connection ~ 7050 1400
-Wire Wire Line
-	7050 1400 6700 1400
+	1    0    0    1
+$EndComp
+Wire Wire Line
+	6700 1400 7450 1400
 $EndSCHEMATC
