File: microsynth/microsynth.kicad_pcb (KiCad board)
At the start: 2 copper layers, 365.8 x 153.7 mm, 273 parts, among them J1 AudioJack3, J2 Conn_01x03_Male, J3 Conn_01x04_Male, J4 Conn_01x04_Male, J5 Conn_01x02_Male, J8 AudioJack2, Q1 BC182, Q2 BC182L, Q3 BC548, Q4 BC212 PNP, Q5 BC212 PNP, Q6 BC548, Q7 BC548, Q8 BC548, Q9 BC548, SW1 SW_DP3T, SW10 SW_SPDT, SW11 SW_SPDT, SW12 SW_DP3T, SW13 SW_DP3T, SW14 SW_SPDT, SW15 SW_SPDT, SW16 SW_SPDT, SW17 SW_SPDT, SW18 SW_SPDT, SW19 SW_SPDT, SW2 SW_Rotary2x6, SW20 SW_SPDT, SW21 SW_Rotary2x6, SW22 SW_SPST, SW3 SW_DP3T, SW4 SW_DP3T, SW5 SW_SPDT, SW6 SW_DP3T, SW7 SW_SPDT, SW8 SW_DP3T, SW9 SW_DP3T, U1 RC4136, U10 LM741, U11 LM741, U12 LM741, U13 LM741, U14 4016, U15 LF351, U16 LM741, U17 LM741, U18 LM741, U19 LM741, U2 LM1458, U20 LM13600, U21 CA3080, U22 4013, U23 LM380N, U3 4011, U4 4016, U5 LF347, U6 LF351, U7 LM741, U8 4001, U9 LM741

Commit message: Copper fill GND
Parts:
- moved C20 0.69 mm to (278.4, 110.6)
Routing:
- net TO_VCO1_R79: track 198.1 -> 206.5 mm
- net TO_D3: track 324.1 -> 332.3 mm
- net Net-(C20-Pad2): track 72.6 -> 64.8 mm
- net Net-(C17-Pad1): track 276.2 -> 282.0 mm
- net LFO_TO_VR20_SLIDER: track 505.1 -> 510.9 mm
- net VCO2_SAW: track 115.3 -> 110.1 mm
- net Net-(R133-Pad1): track 299.5 -> 302.6 mm
- net Net-(R142-Pad2): track 335.6 -> 338.6 mm
- net Net-(R150-Pad1): track 176.7 -> 178.5 mm
- net S5_VCO2: track 322.6 -> 324.2 mm
- net TO_VCA_C26: track 359.9 -> 358.4 mm
- net TO_VCA_C27: track 242.4 -> 241.1 mm
- net Net-(R63-Pad1): track 68.0 -> 66.7 mm
- net Net-(C12-Pad1): track 107.5 -> 108.6 mm
- net KEYBOARD_IC7_PIN_6: track 441.7 -> 440.7 mm
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- added copper zone on B.Cu, net GND
- added copper zone on F.Cu, net GND
Other:
- rule via_min_size: 0.4 -> 0.6

Commit message: Add test points
Parts:
- added TP1: VCF OUT, TestPoint:TestPoint_Pad_D2.0mm, F.Cu at (363.4, 210.9)
- added TP2: NOISE, TestPoint:TestPoint_Pad_D2.0mm, F.Cu at (298.0, 148.8)
- added TP3: VCA OUT, TestPoint:TestPoint_Pad_D2.0mm, F.Cu at (386.9, 172.8)
- added TP4: VCO2, TestPoint:TestPoint_Pad_D2.0mm, F.Cu at (206.8, 220.7)
- added TP5: VCO1, TestPoint:TestPoint_Pad_D2.0mm, F.Cu at (80.0, 191.1)
- added TP6: ADSR, TestPoint:TestPoint_Pad_D2.0mm, F.Cu at (207.1, 152.4)
- SW22: value SW_SPST -> VCO1 ON/OFF
Routing:
- net Net-(D8-Pad2): track 7.74 -> 32.9 mm
- net TO_VCF_IC20_3: track 411.1 -> 430.7 mm
- net LFO_TO_VR20_SLIDER: track 510.9 -> 526.0 mm
- net VCF_OUT: track 28.5 -> 38.3 mm
- net Net-(C29-Pad2): track 6.37 -> 11.2 mm
- net NOISE: track 42.9 -> 47.7 mm
- net Net-(RV19-Pad2): track 49.1 -> 53.6 mm
- net Net-(R142-Pad2): track 338.6 -> 339.3 mm

Commit message: Remove smd footprints, create and assign power/default tracks, tidy up ground planes
Routing:
- net +VSW: track 1365.2 -> 1351.9 mm
- net Net-(R133-Pad1): track 302.6 -> 313.8 mm
- net S5_VCO2: track 324.2 -> 332.5 mm
- net VCO1_SAW1: track 405.7 -> 413.0 mm
- net -VSW: track 1309.1 -> 1302.2 mm
- net TO_D3: track 332.3 -> 338.7 mm
- net Net-(C7-Pad1): track 454.1 -> 457.6 mm
- net ENVELOPE: track 163.6 -> 166.9 mm
- net LFO_TO_VR20_SLIDER: track 526.0 -> 529.0 mm
- net Net-(SW8-Pad3): track 105.7 -> 102.8 mm
- net Net-(C16-Pad2): track 44.3 -> 46.4 mm
- net Net-(C13-Pad2): track 293.9 -> 291.9 mm
- net Net-(C1-Pad1): track 65.0 -> 63.3 mm
- net GND: track 1074.8 -> 1073.1 mm, vias 2 -> 12
- net KEYBOARD_IC7_PIN_6: track 440.7 -> 442.1 mm
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Other:
- net class GND removed
- net class Power added: clearance 0.25, trace_width 1, via_dia 0.8, via_drill 0.4
- net class Rustic removed

Commit message: More ground plane tidy ups
Routing:
- net Net-(Q9-Pad2): track 45.2 -> 25.8 mm
- net TO_VCA_C27: track 241.0 -> 236.0 mm
- net S5_VCO2: track 332.5 -> 337.1 mm
- net GND: track 1073.1 -> 1069.5 mm
- net Net-(C34-Pad1): track 14.1 -> 11.8 mm
- net Net-(Q4-Pad3): track 305.9 -> 308.0 mm
- net TO_RANGE: track 171.4 -> 173.1 mm
- net Net-(C31-Pad2): track 17.6 -> 16.2 mm
- net Net-(R149-Pad2): track 20.8 -> 19.5 mm
- net Net-(C31-Pad1): track 22.4 -> 21.4 mm
- net KEYBOARD_IC7_PIN_6: track 442.1 -> 443.1 mm
- net Net-(R72-Pad1): track 88.3 -> 89.2 mm
- net VCF_OUT: track 38.3 -> 39.2 mm
- net TO_VCA_C26: track 358.4 -> 357.8 mm
Other:
- board text added: "v1.0.0"

Commit message: Update switch footprints with bigger pads
Routing:
- net Net-(RV19-Pad2): track 53.6 -> 50.2 mm
- net Net-(C7-Pad1): track 457.6 -> 455.0 mm
- net Net-(Q3-Pad1): track 75.9 -> 73.7 mm
- net Net-(R133-Pad1): track 313.7 -> 313.0 mm
- net TO_D3: track 338.7 -> 339.3 mm
- net KEYBOARD_IC7_PIN_6: track 443.1 -> 443.7 mm
- net GND: vias 12 -> 14

Commit message: Update switch footprints with bigger pads again
Parts:
- moved R99 2.23 mm to (249.4, 228.1)
- moved R103 0.94 mm to (317.7, 229.5)
- moved R118 0.74 mm to (351.7, 202.3)
Routing:
- net Net-(R140-Pad2): track 228.9 -> 217.7 mm
- net Net-(R133-Pad1): track 313.0 -> 321.0 mm
- net Net-(R77-Pad2): track 413.9 -> 421.1 mm
- net TO_VCF_IC20_3: track 430.7 -> 436.5 mm
- net Net-(SW21-Pad14): track 278.7 -> 283.6 mm
- net TO_VCO1_R79: track 207.0 -> 202.3 mm
- net TO_VCA_C26: track 357.8 -> 361.4 mm
- net S5_VCO2: track 337.2 -> 340.5 mm
- net Net-(RV27-Pad2): track 111.8 -> 114.4 mm
- net Net-(C7-Pad1): track 455.0 -> 457.5 mm
- net Net-(R142-Pad2): track 339.1 -> 337.2 mm
- net LFO_MOD_S16: track 15.6 -> 17.3 mm
- net Net-(SW9-Pad1): track 299.0 -> 297.4 mm
- net VCF_OUT: track 39.2 -> 40.7 mm
- net Net-(RV27-Pad3): track 96.1 -> 94.8 mm
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- removed copper zone on B.Cu, net GND
- removed copper zone on F.Cu, net GND
